File: breakouts/adf4355-3/adf4355-3.kicad_pcb (KiCad board)
At the start: 4 copper layers, 38.2 x 23.5 mm, 57 parts, among them P1 CONN_01X02, P2 CONN_01X06, P3 CONN_01X05, P4 CONN_01X05, P5 CONN_01X05, U1 ADM7150, U2 TCM-63AX+, U3 TCM-63AX+, U4 ADF4355-3, U5 mounting_box, U6 

Commit message: ready to order demod, pcm breakout, booster, and synth
Parts:
- added D1: LED, LEDs:LED_0603, F.Cu at (167.6, 98.2)
- added D2: LED, LEDs:LED_0603, F.Cu at (137.8, 108.3)
- added R4: 1k, Resistors_SMD:R_0402, F.Cu at (164.6, 98.2)
- added R5: 1k, Resistors_SMD:R_0402, B.Cu at (139.8, 106.0)
- U6: value (none) -> TXCO
Routing:
- net GND: track 55.7 -> 87.9 mm, vias 43 -> 45
- net /ADF_LOCK: track 11.5 -> 14.7 mm
- net Net-(D2-Pad1): track 0.00 -> 2.76 mm, vias 0 -> 1
- net Net-(D1-Pad1): track 0.00 -> 1.75 mm
- net /VCC_RF: track 32.2 -> 33.2 mm, vias 12 -> 13
