File: breakouts/pcm2900/pcm2900.sch (KiCad schematic (older format))
At the start: 31 parts, among them P1 USB_OTG, P2 CONN_01X04, P3 CONN_01X03, U1 CONN_SMA, U2 CONN_SMA, U3 pcm2900, Y1 12 MHz

Commit message: added leds to pcm2900, demod, and synth boards. started layout on ti boosterpack control hat
Parts:
- added D1: LED, LEDs:LED_0603, symbol LED
- added R14: 1k, Resistors_SMD:R_0603, symbol R_Small
Connections:
- net GND: now also R14.1
- net at C6.1, R10.2, U3.27 (Vddi)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: now also D1.2 (A)
- new net: D1.1 (K), R14.2
Changed lines of the file:
@@
 $EndComp
 $Comp
-L GND #PWR01
+L GND #PWR11
 U 1 1 56DDC904
 P 5900 5550
-F 0 "#PWR01" H 5900 5300 50  0001 C CNN
+F 0 "#PWR11" H 5900 5300 50  0001 C CNN
 F 1 "GND" H 5900 5400 50  0000 C CNN
 F 2 "" H 5900 5550 50  0000 C CNN
@@
 NoConn ~ 5250 3650
 $Comp
-L GND #PWR02
+L GND #PWR8
 U 1 1 56DDCAAD
 P 5350 3550
-F 0 "#PWR02" H 5350 3300 50  0001 C CNN
+F 0 "#PWR8" H 5350 3300 50  0001 C CNN
 F 1 "GND" H 5350 3400 50  0000 C CNN
 F 2 "" H 5350 3550 50  0000 C CNN
@@
 $EndComp
 $Comp
-L GND #PWR03
+L GND #PWR9
 U 1 1 56DDCB3E
 P 5350 4350
-F 0 "#PWR03" H 5350 4100 50  0001 C CNN
+F 0 "#PWR9" H 5350 4100 50  0001 C CNN
 F 1 "GND" H 5350 4200 50  0000 C CNN
 F 2 "" H 5350 4350 50  0000 C CNN
@@
 NoConn ~ 6200 4350
 $Comp
-L GND #PWR04
+L GND #PWR14
 U 1 1 56DDD0B1
 P 7650 3950
-F 0 "#PWR04" H 7650 3700 50  0001 C CNN
+F 0 "#PWR14" H 7650 3700 50  0001 C CNN
 F 1 "GND" H 7650 3800 50  0000 C CNN
 F 2 "" H 7650 3950 50  0000 C CNN
@@
 	7600 3850 7600 3000
 Wire Wire Line
-	7600 3000 5650 3000
+	5650 3000 8200 3000
 Wire Wire Line
 	5650 3000 5650 3250
@@
 NoConn ~ 7400 4050
 $Comp
-L GND #PWR05
+L GND #PWR15
 U 1 1 56DDD151
 P 7650 4350
-F 0 "#PWR05" H 7650 4100 50  0001 C CNN
+F 0 "#PWR15" H 7650 4100 50  0001 C CNN
 F 1 "GND" H 7650 4200 50  0000 C CNN
 F 2 "" H 7650 4350 50  0000 C CNN
@@
 	8900 4700 9000 4700
 $Comp
-L GND #PWR06
+L GND #PWR21
 U 1 1 56DDD82A
 P 9000 4400
-F 0 "#PWR06" H 9000 4150 50  0001 C CNN
+F 0 "#PWR21" H 9000 4150 50  0001 C CNN
 F 1 "GND" H 9000 4250 50  0000 C CNN
 F 2 "" H 9000 4400 50  0000 C CNN
@@
 $EndComp
 $Comp
-L GND #PWR07
+L GND #PWR22
 U 1 1 56DDD856
 P 9000 4700
-F 0 "#PWR07" H 9000 4450 50  0001 C CNN
+F 0 "#PWR22" H 9000 4450 50  0001 C CNN
 F 1 "GND" H 9000 4550 50  0000 C CNN
 F 2 "" H 9000 4700 50  0000 C CNN
@@
 	7400 4850 7550 4850
 $Comp
-L GND #PWR08
+L GND #PWR17
 U 1 1 56DDDAD7
 P 7850 4750
-F 0 "#PWR08" H 7850 4500 50  0001 C CNN
+F 0 "#PWR17" H 7850 4500 50  0001 C CNN
 F 1 "GND" H 7850 4600 50  0000 C CNN
 F 2 "" H 7850 4750 50  0000 C CNN
@@
 	8200 5050 8350 5050
 $Comp
-L GND #PWR09
+L GND #PWR19
 U 1 1 56DDE2A8
 P 8250 5250
-F 0 "#PWR09" H 8250 5000 50  0001 C CNN
+F 0 "#PWR19" H 8250 5000 50  0001 C CNN
 F 1 "GND" H 8250 5100 50  0000 C CNN
 F 2 "" H 8250 5250 50  0000 C CNN
@@
 $EndComp
 $Comp
-L GND #PWR010
+L GND #PWR2
 U 1 1 56DDED49
 P 850 5650
-F 0 "#PWR010" H 850 5400 50  0001 C CNN
+F 0 "#PWR2" H 850 5400 50  0001 C CNN
 F 1 "GND" H 850 5500 50  0000 C CNN
 F 2 "" H 850 5650 50  0000 C CNN
@@
 $EndComp
 $Comp
-L GND #PWR011
+L GND #PWR1
 U 1 1 56DDF206
 P 800 6850
-F 0 "#PWR011" H 800 6600 50  0001 C CNN
+F 0 "#PWR1" H 800 6600 50  0001 C CNN
 F 1 "GND" H 800 6700 50  0000 C CNN
 F 2 "" H 800 6850 50  0000 C CNN
@@
 	2300 5050 2300 5200
 $Comp
-L GND #PWR012
+L GND #PWR4
 U 1 1 56DDFF12
 P 1800 5600
-F 0 "#PWR012" H 1800 5350 50  0001 C CNN
+F 0 "#PWR4" H 1800 5350 50  0001 C CNN
 F 1 "GND" H 1800 5450 50  0000 C CNN
 F 2 "" H 1800 5600 50  0000 C CNN
@@
 	1800 5600 1800 5400
 $Comp
-L GND #PWR013
+L GND #PWR6
 U 1 1 56DDFFD5
 P 2300 5600
-F 0 "#PWR013" H 2300 5350 50  0001 C CNN
+F 0 "#PWR6" H 2300 5350 50  0001 C CNN
 F 1 "GND" H 2300 5450 50  0000 C CNN
 F 2 "" H 2300 5600 50  0000 C CNN
@@
 	2250 6250 2250 6400
 $Comp
-L GND #PWR014
+L GND #PWR3
 U 1 1 56DE0306
 P 1750 6800
-F 0 "#PWR014" H 1750 6550 50  0001 C CNN
+F 0 "#PWR3" H 1750 6550 50  0001 C CNN
 F 1 "GND" H 1750 6650 50  0000 C CNN
 F 2 "" H 1750 6800 50  0000 C CNN
@@
 	1750 6800 1750 6600
 $Comp
-L GND #PWR015
+L GND #PWR5
 U 1 1 56DE030D
 P 2250 6800
-F 0 "#PWR015" H 2250 6550 50  0001 C CNN
+F 0 "#PWR5" H 2250 6550 50  0001 C CNN
 F 1 "GND" H 2250 6650 50  0000 C CNN
 F 2 "" H 2250 6800 50  0000 C CNN
@@
 VCOM
 $Comp
-L GND #PWR016
+L GND #PWR7
 U 1 1 56DE0C67
 P 4600 5900
-F 0 "#PWR016" H 4600 5650 50  0001 C CNN
+F 0 "#PWR7" H 4600 5650 50  0001 C CNN
 F 1 "GND" H 4600 5750 50  0000 C CNN
 F 2 "" H 4600 5900 50  0000 C CNN
@@
 $EndComp
 $Comp
-L GND #PWR017
+L GND #PWR16
 U 1 1 56DE1AE9
 P 7800 3700
-F 0 "#PWR017" H 7800 3450 50  0001 C CNN
+F 0 "#PWR16" H 7800 3450 50  0001 C CNN
 F 1 "GND" H 7800 3550 50  0000 C CNN
 F 2 "" H 7800 3700 50  0000 C CNN
@@
 	5350 4650 5350 5200
 $Comp
-L GND #PWR018
+L GND #PWR10
 U 1 1 56DDD5DA
 P 5350 5550
-F 0 "#PWR018" H 5350 5300 50  0001 C CNN
+F 0 "#PWR10" H 5350 5300 50  0001 C CNN
 F 1 "GND" H 5350 5400 50  0000 C CNN
 F 2 "" H 5350 5550 50  0000 C CNN
@@
 	5350 5550 5350 5400
 $Comp
-L GND #PWR019
+L GND #PWR13
 U 1 1 56DDD6CE
 P 6050 4750
-F 0 "#PWR019" H 6050 4500 50  0001 C CNN
+F 0 "#PWR13" H 6050 4500 50  0001 C CNN
 F 1 "GND" H 6050 4600 50  0000 C CNN
 F 2 "" H 6050 4750 50  0000 C CNN
@@
 	6050 4750 6200 4750
 $Comp
-L GND #PWR020
+L GND #PWR12
 U 1 1 56DDD8D5
 P 6050 4050
-F 0 "#PWR020" H 6050 3800 50  0001 C CNN
+F 0 "#PWR12" H 6050 3800 50  0001 C CNN
 F 1 "GND" H 6050 3900 50  0000 C CNN
 F 2 "" H 6050 4050 50  0000 C CNN
@@
 $EndComp
 $Comp
-L GND #PWR021
+L GND #PWR20
 U 1 1 56DDDE8F
 P 8300 4250
-F 0 "#PWR021" H 8300 4000 50  0001 C CNN
+F 0 "#PWR20" H 8300 4000 50  0001 C CNN
 F 1 "GND" H 8300 4100 50  0000 C CNN
 F 2 "" H 8300 4250 50  0000 C CNN
@@
 Text Label 4650 4850 2    60   ~ 0
 SMA_Q
+$Comp
+L LED D1
+U 1 1 56DE6465
+P 8200 3300
+F 0 "D1" H 8200 3400 50  0000 C CNN
+F 1 "LED" H 8200 3200 50  0000 C CNN
+F 2 "LEDs:LED_0603" H 8200 3300 50  0001 C CNN
+F 3 "" H 8200 3300 50  0000 C CNN
+	1    8200 3300
+	0    -1   -1   0
+$EndComp
+$Comp
+L R_Small R14
+U 1 1 56DE66A2
+P 8200 3700
+F 0 "R14" V 8150 3500 50  0000 L CNN
+F 1 "1k" V 8150 3800 50  0000 L CNN
+F 2 "Resistors_SMD:R_0603" H 8200 3700 50  0001 C CNN
+F 3 "" H 8200 3700 50  0000 C CNN
+	1    8200 3700
+	-1   0    0    1
+$EndComp
+$Comp
+L GND #PWR18
+U 1 1 56DE68B1
+P 8200 3900
+F 0 "#PWR18" H 8200 3650 50  0001 C CNN
+F 1 "GND" H 8200 3750 50  0000 C CNN
+F 2 "" H 8200 3900 50  0000 C CNN
+F 3 "" H 8200 3900 50  0000 C CNN
+	1    8200 3900
+	1    0    0    -1
+$EndComp
+Wire Wire Line
+	8200 3800 8200 3900
+Wire Wire Line
+	8200 3500 8200 3600
+Wire Wire Line
+	8200 3000 8200 3100
+Connection ~ 7600 3000
 $EndSCHEMATC

Commit message: started variable attenuator, revised synth, and added power splittert to detect board
Parts:
- R14: value 1k -> 1k5
Changed lines of the file:
@@
 LIBS:rf_crossbar
 LIBS:scbd-16-63
-LIBS:sma_keepout
 LIBS:tcm-63ax+
 LIBS:txco
@@
 $EndComp
 $Comp
-L GND #PWR11
+L GND #PWR01
 U 1 1 56DDC904
 P 5900 5550
-F 0 "#PWR11" H 5900 5300 50  0001 C CNN
+F 0 "#PWR01" H 5900 5300 50  0001 C CNN
 F 1 "GND" H 5900 5400 50  0000 C CNN
 F 2 "" H 5900 5550 50  0000 C CNN
@@
 NoConn ~ 5250 3650
 $Comp
-L GND #PWR8
+L GND #PWR02
 U 1 1 56DDCAAD
 P 5350 3550
-F 0 "#PWR8" H 5350 3300 50  0001 C CNN
+F 0 "#PWR02" H 5350 3300 50  0001 C CNN
 F 1 "GND" H 5350 3400 50  0000 C CNN
 F 2 "" H 5350 3550 50  0000 C CNN
@@
 $EndComp
 $Comp
-L GND #PWR9
+L GND #PWR03
 U 1 1 56DDCB3E
 P 5350 4350
-F 0 "#PWR9" H 5350 4100 50  0001 C CNN
+F 0 "#PWR03" H 5350 4100 50  0001 C CNN
 F 1 "GND" H 5350 4200 50  0000 C CNN
 F 2 "" H 5350 4350 50  0000 C CNN
@@
 NoConn ~ 6200 4350
 $Comp
-L GND #PWR14
+L GND #PWR04
 U 1 1 56DDD0B1
 P 7650 3950
-F 0 "#PWR14" H 7650 3700 50  0001 C CNN
+F 0 "#PWR04" H 7650 3700 50  0001 C CNN
 F 1 "GND" H 7650 3800 50  0000 C CNN
 F 2 "" H 7650 3950 50  0000 C CNN
@@
 NoConn ~ 7400 4050
 $Comp
-L GND #PWR15
+L GND #PWR05
 U 1 1 56DDD151
 P 7650 4350
-F 0 "#PWR15" H 7650 4100 50  0001 C CNN
+F 0 "#PWR05" H 7650 4100 50  0001 C CNN
 F 1 "GND" H 7650 4200 50  0000 C CNN
 F 2 "" H 7650 4350 50  0000 C CNN
@@
 	8900 4700 9000 4700
 $Comp
-L GND #PWR21
+L GND #PWR06
 U 1 1 56DDD82A
 P 9000 4400
-F 0 "#PWR21" H 9000 4150 50  0001 C CNN
+F 0 "#PWR06" H 9000 4150 50  0001 C CNN
 F 1 "GND" H 9000 4250 50  0000 C CNN
 F 2 "" H 9000 4400 50  0000 C CNN
@@
 $EndComp
 $Comp
-L GND #PWR22
+L GND #PWR07
 U 1 1 56DDD856
 P 9000 4700
-F 0 "#PWR22" H 9000 4450 50  0001 C CNN
+F 0 "#PWR07" H 9000 4450 50  0001 C CNN
 F 1 "GND" H 9000 4550 50  0000 C CNN
 F 2 "" H 9000 4700 50  0000 C CNN
@@
 	7400 4850 7550 4850
 $Comp
-L GND #PWR17
+L GND #PWR08
 U 1 1 56DDDAD7
 P 7850 4750
-F 0 "#PWR17" H 7850 4500 50  0001 C CNN
+F 0 "#PWR08" H 7850 4500 50  0001 C CNN
 F 1 "GND" H 7850 4600 50  0000 C CNN
 F 2 "" H 7850 4750 50  0000 C CNN
@@
 	8200 5050 8350 5050
 $Comp
-L GND #PWR19
+L GND #PWR09
 U 1 1 56DDE2A8
 P 8250 5250
-F 0 "#PWR19" H 8250 5000 50  0001 C CNN
+F 0 "#PWR09" H 8250 5000 50  0001 C CNN
 F 1 "GND" H 8250 5100 50  0000 C CNN
 F 2 "" H 8250 5250 50  0000 C CNN
@@
 $EndComp
 $Comp
-L GND #PWR2
+L GND #PWR010
 U 1 1 56DDED49
 P 850 5650
-F 0 "#PWR2" H 850 5400 50  0001 C CNN
+F 0 "#PWR010" H 850 5400 50  0001 C CNN
 F 1 "GND" H 850 5500 50  0000 C CNN
 F 2 "" H 850 5650 50  0000 C CNN
@@
 $EndComp
 $Comp
-L GND #PWR1
+L GND #PWR011
 U 1 1 56DDF206
 P 800 6850
-F 0 "#PWR1" H 800 6600 50  0001 C CNN
+F 0 "#PWR011" H 800 6600 50  0001 C CNN
 F 1 "GND" H 800 6700 50  0000 C CNN
 F 2 "" H 800 6850 50  0000 C CNN
@@
 	2300 5050 2300 5200
 $Comp
-L GND #PWR4
+L GND #PWR012
 U 1 1 56DDFF12
 P 1800 5600
-F 0 "#PWR4" H 1800 5350 50  0001 C CNN
+F 0 "#PWR012" H 1800 5350 50  0001 C CNN
 F 1 "GND" H 1800 5450 50  0000 C CNN
 F 2 "" H 1800 5600 50  0000 C CNN
@@
 	1800 5600 1800 5400
 $Comp
-L GND #PWR6
+L GND #PWR013
 U 1 1 56DDFFD5
 P 2300 5600
-F 0 "#PWR6" H 2300 5350 50  0001 C CNN
+F 0 "#PWR013" H 2300 5350 50  0001 C CNN
 F 1 "GND" H 2300 5450 50  0000 C CNN
 F 2 "" H 2300 5600 50  0000 C CNN
@@
 	2250 6250 2250 6400
 $Comp
-L GND #PWR3
+L GND #PWR014
 U 1 1 56DE0306
 P 1750 6800
-F 0 "#PWR3" H 1750 6550 50  0001 C CNN
+F 0 "#PWR014" H 1750 6550 50  0001 C CNN
 F 1 "GND" H 1750 6650 50  0000 C CNN
 F 2 "" H 1750 6800 50  0000 C CNN
@@
 	1750 6800 1750 6600
 $Comp
-L GND #PWR5
+L GND #PWR015
 U 1 1 56DE030D
 P 2250 6800
-F 0 "#PWR5" H 2250 6550 50  0001 C CNN
+F 0 "#PWR015" H 2250 6550 50  0001 C CNN
 F 1 "GND" H 2250 6650 50  0000 C CNN
 F 2 "" H 2250 6800 50  0000 C CNN
@@
 VCOM
 $Comp
-L GND #PWR7
+L GND #PWR016
 U 1 1 56DE0C67
 P 4600 5900
-F 0 "#PWR7" H 4600 5650 50  0001 C CNN
+F 0 "#PWR016" H 4600 5650 50  0001 C CNN
 F 1 "GND" H 4600 5750 50  0000 C CNN
 F 2 "" H 4600 5900 50  0000 C CNN
@@
 $EndComp
 $Comp
-L GND #PWR16
+L GND #PWR017
 U 1 1 56DE1AE9
 P 7800 3700
-F 0 "#PWR16" H 7800 3450 50  0001 C CNN
+F 0 "#PWR017" H 7800 3450 50  0001 C CNN
 F 1 "GND" H 7800 3550 50  0000 C CNN
 F 2 "" H 7800 3700 50  0000 C CNN
@@
 	5350 4650 5350 5200
 $Comp
-L GND #PWR10
+L GND #PWR018
 U 1 1 56DDD5DA
 P 5350 5550
-F 0 "#PWR10" H 5350 5300 50  0001 C CNN
+F 0 "#PWR018" H 5350 5300 50  0001 C CNN
 F 1 "GND" H 5350 5400 50  0000 C CNN
 F 2 "" H 5350 5550 50  0000 C CNN
@@
 	5350 5550 5350 5400
 $Comp
-L GND #PWR13
+L GND #PWR019
 U 1 1 56DDD6CE
 P 6050 4750
-F 0 "#PWR13" H 6050 4500 50  0001 C CNN
+F 0 "#PWR019" H 6050 4500 50  0001 C CNN
 F 1 "GND" H 6050 4600 50  0000 C CNN
 F 2 "" H 6050 4750 50  0000 C CNN
@@
 	6050 4750 6200 4750
 $Comp
-L GND #PWR12
+L GND #PWR020
 U 1 1 56DDD8D5
 P 6050 4050
-F 0 "#PWR12" H 6050 3800 50  0001 C CNN
+F 0 "#PWR020" H 6050 3800 50  0001 C CNN
 F 1 "GND" H 6050 3900 50  0000 C CNN
 F 2 "" H 6050 4050 50  0000 C CNN
@@
 $EndComp
 $Comp
-L GND #PWR20
+L GND #PWR021
 U 1 1 56DDDE8F
 P 8300 4250
-F 0 "#PWR20" H 8300 4000 50  0001 C CNN
+F 0 "#PWR021" H 8300 4000 50  0001 C CNN
 F 1 "GND" H 8300 4100 50  0000 C CNN
 F 2 "" H 8300 4250 50  0000 C CNN
@@
 P 8200 3700
 F 0 "R14" V 8150 3500 50  0000 L CNN
-F 1 "1k" V 8150 3800 50  0000 L CNN
+F 1 "1k5" V 8150 3800 50  0000 L CNN
 F 2 "Resistors_SMD:R_0603" H 8200 3700 50  0001 C CNN
 F 3 "" H 8200 3700 50  0000 C CNN
@@
 $EndComp
 $Comp
-L GND #PWR18
+L GND #PWR022
 U 1 1 56DE68B1
 P 8200 3900
-F 0 "#PWR18" H 8200 3650 50  0001 C CNN
+F 0 "#PWR022" H 8200 3650 50  0001 C CNN
 F 1 "GND" H 8200 3750 50  0000 C CNN
 F 2 "" H 8200 3900 50  0000 C CNN
