File: breakouts/synth/synth.sch (KiCad schematic (older format))
At the start: 48 parts

Commit message: started and finished variable attenuator layout
Parts:
- removed U? (x2): CONN_SMA, symbol CONN_SMA
- added C29, C31, C33, C35, C37, C39: 30 pF, Capacitors_SMD:C_0402, symbol C_Small
- added C30, C32, C34, C36, C38, C40: 100 nF, Capacitors_SMD:C_0402, symbol C_Small
- added L1, L2: 18 nF, Resistors_SMD:R_0402, symbol L_Small
- added P1: CONN_01X07, Pin_Headers:Pin_Header_Straight_1x07, symbol CONN_01X07
- added R12, R13, R14, R15, R16: R_Small, Resistors_SMD:R_0402, symbol R_Small
- added R18, R19, R20, R21, R22, R23, R24, R25, R26, R27: 49.9, Resistors_SMD:R_0402, symbol R_Small
- added U4, U5, U7: CONN_SMA, vna_footprints:732512200_SMA, symbol CONN_SMA
- C1, C10, C11, C13, C16, C17, C18, C19, C20, C23, C24, C25, C28, C3, C5, C7, C9: renamed from C?; footprint (none) -> Capacitors_SMD:C_0402
- C12, C2, C21, C22, C26, C27, C4, C6, C8: renamed from C?; footprint (none) -> Capacitors_SMD:C_0805
- C14: renamed from C?; value 100 nF -> 1 uF; footprint (none) -> Capacitors_SMD:C_0402
- C15: renamed from C?; value .047 uF -> 47 nF; footprint (none) -> Capacitors_SMD:C_0402
- D1, D2: renamed from D?; footprint (none) -> LEDs:LED_0603
- R1, R10, R11, R17, R2, R3, R4, R5, R6, R7, R8, R9: renamed from R?; footprint (none) -> Resistors_SMD:R_0402
- U1, U6: renamed from U?; footprint (none) -> vna_footprints:732512200_SMA
- U2: renamed from U?; footprint (none) -> vna_footprints:crystal_FA238-TSX3225
- U3: renamed from U?; footprint (none) -> Housings_DFN_QFN:QFN-40-1EP_6x6mm_Pitch0.5mm
Connections:
- net VCC is gone; now on net GND: C1.1, C16.2, C18.1, C2.1, C20.2, C25.1, C28.2, C3.1, C4.1, C5.1, C6.1, C7.1, C8.1, C9.1, D2.2 (A), R1.2, U2.4 (VCC), U3.11 (VccCP), U3.15 (VccMASH), U3.21 (VccBUF), U3.26 (VccVCO2), U3.37 (VccVCO)
- net CE: now also P1.7 (P7), R12.2
- net CSB: now also R13.1
- net GND: now also C29.1, C29.2, C30.1, C30.2, C35.1, C35.2, C36.1, C36.2, L1.2, L2.1, P1.1 (P1), P1.2 (P2), R12.1, R18.1, R19.2, R22.1, R23.1, R26.1, R27.1, U4.2 (GND), U4.3 (GND), U4.4 (GND), U4.5 (GND), U5.2 (GND), U5.3 (GND), U5.4 (GND), U5.5 (GND), U7.2 (GND), U7.3 (GND), U7.4 (GND), U7.5 (GND)
- net MUXout: now also R14.1
- net SCK: now also R16.1
- net SDI: now also R15.1
- net RFoutBP: now reaches U3.18 (RFoutBP)
- net RFoutBP: now also C37.2, C38.2, R18.2
- net RFoutBM: now reaches U3.19 (RFoutBM)
- net RFoutBM: now also C39.2, C40.2, R19.1
- net RFoutAM: now reaches U3.22 (RFoutAM)
- net RFoutAM: now also C31.2, C32.2, L1.1
- net RFoutAP: now reaches U3.23 (RFoutAP)
- net RFoutAP: now also C33.2, C34.2, L2.2
- net at U6.1 (RF): now also C37.1, C38.1, R26.2
- new net: P1.6 (P6), R13.2
- new net: P1.5 (P5), R14.2
- new net: P1.4 (P4), R15.2
- new net: P1.3 (P3), R16.2
- new net: C39.1, C40.1, R27.2, U7.1 (RF)
- new net: R24.2, U4.1 (RF)
- new net: C33.1, C34.1, R21.1
- new net: R20.2, R22.2, R24.1
- new net: R21.2, R23.2, R25.1
- new net: R25.2, U5.1 (RF)
- new net: C31.1, C32.1, R20.1
Other:
- note added: "6 dBm in"
- moved on the sheet: U6

Commit message: stared on control of other rf modules..
Parts:
- added U8: mounting_box, vna_footprints:POMONA_2400BOX, symbol mounting_box
- C12, C2, C21, C22, C26, C27, C4, C6, C8: footprint Capacitors_SMD:C_0805 -> Capacitors_SMD:C_0603
- R12, R13, R14, R15, R16, R6, R7, R8: value R_Small -> 1k
- R2, R4: value R_Small -> DNP
- R3, R5: value R_Small -> 0
Connections:
- net GND: no longer C1.1, C16.2, C18.1, C2.1, C20.2, C25.1, C28.2, C29.2, C3.1, C30.2, C35.2, C36.2, C4.1, C5.1, C6.1, C7.1, C8.1, C9.1, D2.2 (A), L1.2, L2.1, P1.2 (P2), R1.2, R12.1, R18.1, R19.2, U2.4 (VCC), U3.11 (VccCP), U3.15 (VccMASH), U3.21 (VccBUF), U3.26 (VccVCO2), U3.37 (VccVCO)
- net RFoutAM: now also C33.2, C34.2, L2.2; no longer C31.2, C32.2, L1.1
- net RFoutAP: now also C31.2, C32.2, L1.1; no longer C33.2, C34.2, L2.2
- net RFoutBM: now also C37.2, C38.2, R18.2; no longer C39.2, C40.2, R19.1
- net RFoutBP: now also C39.2, C40.2, R19.1; no longer C37.2, C38.2, R18.2
- net VCC: now reaches C13.2, U3.7 (VccDIG)
- net VCC: now also C1.1, C16.2, C18.1, C2.1, C20.2, C25.1, C28.2, C29.2, C3.1, C30.2, C35.2, C36.2, C4.1, C5.1, C6.1, C7.1, C8.1, C9.1, D2.2 (A), L1.2, L2.1, P1.2 (P2), R1.2, R12.1, R18.1, R19.2, U2.4 (VCC), U3.11 (VccCP), U3.15 (VccMASH), U3.21 (VccBUF), U3.26 (VccVCO2), U3.37 (VccVCO)
