File: breakouts/attenuator/attenuator.kicad_pcb (KiCad board)
At the start: 4 copper layers, 36.8 x 24.1 mm, 37 parts, among them P1 CONN_01X08, U1 CONN_SMA, U2 LTC1983, U3 HMC424, U4 CONN_SMA, U5 74HC04, U6 mounting_box

Commit message: changed sma connectors on amp board to edge launch, trimmed excess ground plane
Changed lines of the file:
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@@
   (general
     (links 82)
-    (no_connects 34)
+    (no_connects 0)
     (area 121.814999 85.883 175.365001 123.575)
     (thickness 1.6)
@@
     (effects (font (size 1 1) (thickness 0.25)) (justify left))
   )
-  (gr_circle (center 132.334 101.854) (end 132.08 101.854) (layer F.SilkS) (width 0.2))
+  (gr_circle (center 128.905 107.315) (end 128.651 107.315) (layer F.SilkS) (width 0.2))
   (gr_circle (center 143.764 95.504) (end 143.51 95.504) (layer F.SilkS) (width 0.2))
   (gr_text "variable attenuator r0" (at 150.622 93.98) (layer F.SilkS)
