File: hardware/switch_demod/adc.sch (KiCad schematic (older format))
At the start: 64 parts

Commit message: a little more work on demod/adc board
Parts:
- JP701: renamed from JP?; footprint (none) -> Resistors_SMD:R_1206
- gave numbers to parts that had none: 63
Connections:
- net ADC_I_M renamed ADC_I_N
- net ADC_Q_M renamed ADC_Q_N
