File: hardware/switch_demod/connectors_control_pow.sch (KiCad schematic (older format))
At the start: 0 parts

Commit message: a little more work on demod/adc board
Parts:
- added C901: 100 uF, Capacitors_SMD:C_1210, symbol CP_Small
- added D901: RED, LEDs:LED_0603, symbol LED
- added F901: PTC, Resistors_SMD:R_1210, symbol FUSE
- added H901, H902, H903, H904: MOUNTING_HOLE, Mounting_Holes:MountingHole_2-7mm, symbol MOUNTING_HOLE
- added L901: FERRITE CHIP, Resistors_SMD:R_0805, symbol INDUCTOR_SMALL
- added P901: CONN_01X02, Terminal_Blocks:TerminalBlock_Pheonix_PT-3.5mm_2pol, symbol CONN_01X02
- added Q901: DMG2305UX, TO_SOT_Packages_SMD:SOT-23, symbol Q_PMOS_GSD
- added R901: 1k, Resistors_SMD:R_0402, symbol R_Small
- added SW?: SWITCH_INV, symbol SWITCH_INV
- added U901: CONN_SMA_2GND, vna_footprints:142-0721-882_sma_cutout, symbol CONN_SMA_2GND
Connections:
- new net: F901.2, P901.1 (P1), SW?.3
- new net: F901.1, Q901.3 (D)
- new net: L901.2, Q901.2 (S)
- new net: Q901.1 (G), SW?.2
- new net: D901.1 (K), R901.1
- new net +5V: C901.1, D901.2 (A), L901.1
- new net GND: C901.2, P901.2 (P2), R901.2, SW?.1, U901.2 (GND), U901.3 (GND)
- new net SYNTH_IN: U901.1 (RF)
Other:
- note added: "TODO: add fuse, reverse polarity, power led"
- note added: "TODO: simulate switch\n"
- note added: "TODO:\ncreate beaglebone header symbol\ncheck io voltages, add buffers?\nadd ADC clock input\nadd adc input netlist length constraints"
