File: hardware/switch_demod/splitter_lo.sch (KiCad schematic (older format))
At the start: 1 part

Commit message: a little more work on demod/adc board
Parts:
- U501: renamed from U?; footprint (none) -> vna_footprints:PS1608
Changed lines of the file:
@@
 $Descr A4 11693 8268
 encoding utf-8
-Sheet 6 9
+Sheet 5 9
 Title ""
 Date ""
@@
 $EndDescr
 $Comp
-L PWR_SPLITTER U?
+L PWR_SPLITTER U501
 U 1 1 574CDAE3
 P 6000 3400
-F 0 "U?" H 5600 3800 60  0000 C CNN
+F 0 "U501" H 5600 3800 60  0000 C CNN
 F 1 "PWR_SPLITTER" H 5850 3900 60  0000 C CNN
-F 2 "" H 6000 3400 60  0000 C CNN
+F 2 "vna_footprints:PS1608" H 6000 3400 60  0001 C CNN
 F 3 "" H 6000 3400 60  0000 C CNN
 	1    6000 3400
@@
 $EndComp
 $Comp
-L GND #PWR?
+L GND #PWR053
 U 1 1 574CDAE4
 P 5950 4000
-F 0 "#PWR?" H 5950 3750 50  0001 C CNN
+F 0 "#PWR053" H 5950 3750 50  0001 C CNN
 F 1 "GND" H 5950 3850 50  0000 C CNN
 F 2 "" H 5950 4000 50  0000 C CNN
