File: breakouts/switch_breakout/switch_breakout.sch (KiCad schematic (older format))
At the start: 11 parts, among them P1 CONN_01X03, U1 CONN_SMA, U2 CONN_SMA, U3 PE42521, U4 CONN_SMA, U5 mounting_box

Commit message: finished bias module, modified mixer, splitter, and switch sma connector footprints
Parts:
- removed U1, U2, U4: CONN_SMA, vna_footprints:732511150_sma, symbol CONN_SMA
- removed U5: mounting_box, vna_footprints:POMONA_2400BOX, symbol mounting_box
- added U101, U102, U103: CONN_SMA_2GND, vna_footprints:142-0721-882_sma_cutout, symbol CONN_SMA_2GND
Connections:
- net GND: now also U101.2 (GND), U101.3 (GND), U102.2 (GND), U102.3 (GND), U103.2 (GND), U103.3 (GND)
- net at C5.1: now also U103.1 (RF)
- net at C2.1: now also U102.1 (RF)
- net at C1.1: now also U101.1 (RF)
Changed lines of the file:
@@
 LIBS:conn_sma
 LIBS:mounting_box
+LIBS:conn_sma_2gnd
 LIBS:switch_breakout-cache
 EELAYER 25 0
@@
 	0    1    1    0
 $EndComp
-$Comp
-L CONN_SMA U4
-U 1 1 56AEE9D4
-P 9100 4650
-F 0 "U4" H 8750 4850 60  0000 C CNN
-F 1 "CONN_SMA" H 8950 5000 60  0000 C CNN
-F 2 "vna_footprints:732511150_sma" H 9100 4650 60  0001 C CNN
-F 3 "" H 9100 4650 60  0000 C CNN
-	1    9100 4650
-	1    0    0    -1
-$EndComp
-$Comp
-L GND #PWR01
-U 1 1 56AEEAAA
-P 9100 5350
-F 0 "#PWR01" H 9100 5100 50  0001 C CNN
-F 1 "GND" H 9100 5200 50  0000 C CNN
-F 2 "" H 9100 5350 50  0000 C CNN
-F 3 "" H 9100 5350 50  0000 C CNN
-	1    9100 5350
-	1    0    0    -1
-$EndComp
-Wire Wire Line
-	8950 5100 8950 5250
-Wire Wire Line
-	8950 5250 9250 5250
-Wire Wire Line
-	9250 5250 9250 5100
-Wire Wire Line
-	9150 5100 9150 5250
-Connection ~ 9150 5250
-Wire Wire Line
-	9050 5100 9050 5250
-Connection ~ 9050 5250
-Wire Wire Line
-	9100 5250 9100 5350
-Connection ~ 9100 5250
-Wire Wire Line
-	8350 4650 8550 4650
+Wire Wire Line
+	8350 4650 8750 4650
 Wire Wire Line
 	3550 3350 6300 3350
@@
 	0    -1   1    0
 $EndComp
-$Comp
-L CONN_SMA U2
-U 1 1 56AEF263
-P 2600 5750
-F 0 "U2" H 2250 5950 60  0000 C CNN
-F 1 "CONN_SMA" H 2450 6100 60  0000 C CNN
-F 2 "vna_footprints:732511150_sma" H 2600 5750 60  0001 C CNN
-F 3 "" H 2600 5750 60  0000 C CNN
-	1    2600 5750
-	-1   0    0    -1
-$EndComp
-$Comp
-L GND #PWR02
-U 1 1 56AEF269
-P 2600 6450
-F 0 "#PWR02" H 2600 6200 50  0001 C CNN
-F 1 "GND" H 2600 6300 50  0000 C CNN
-F 2 "" H 2600 6450 50  0000 C CNN
-F 3 "" H 2600 6450 50  0000 C CNN
-	1    2600 6450
-	-1   0    0    -1
-$EndComp
-Wire Wire Line
-	2750 6200 2750 6350
-Wire Wire Line
-	2750 6350 2450 6350
-Wire Wire Line
-	2450 6350 2450 6200
-Wire Wire Line
-	2550 6200 2550 6350
-Connection ~ 2550 6350
-Wire Wire Line
-	2650 6200 2650 6350
-Connection ~ 2650 6350
-Wire Wire Line
-	2600 6350 2600 6450
-Connection ~ 2600 6350
 Wire Wire Line
 	3350 5750 3150 5750
@@
 	6300 5750 6300 5350
 $Comp
-L GND #PWR03
+L GND #PWR111
 U 1 1 56AEF357
 P 6400 5450
-F 0 "#PWR03" H 6400 5200 50  0001 C CNN
+F 0 "#PWR111" H 6400 5200 50  0001 C CNN
 F 1 "GND" H 6400 5300 50  0000 C CNN
 F 2 "" H 6400 5450 50  0000 C CNN
@@
 $EndComp
 $Comp
-L GND #PWR04
+L GND #PWR113
 U 1 1 56AEF39E
 P 6500 5450
-F 0 "#PWR04" H 6500 5200 50  0001 C CNN
+F 0 "#PWR113" H 6500 5200 50  0001 C CNN
 F 1 "GND" H 6500 5300 50  0000 C CNN
 F 2 "" H 6500 5450 50  0000 C CNN
@@
 $EndComp
 $Comp
-L GND #PWR05
+L GND #PWR109
 U 1 1 56AEF4BB
 P 6200 5450
-F 0 "#PWR05" H 6200 5200 50  0001 C CNN
+F 0 "#PWR109" H 6200 5200 50  0001 C CNN
 F 1 "GND" H 6200 5300 50  0000 C CNN
 F 2 "" H 6200 5450 50  0000 C CNN
@@
 	6500 5450 6500 5350
 $Comp
-L GND #PWR06
+L GND #PWR112
 U 1 1 56AEF535
 P 6500 3900
-F 0 "#PWR06" H 6500 3650 50  0001 C CNN
+F 0 "#PWR112" H 6500 3650 50  0001 C CNN
 F 1 "GND" H 6500 3750 50  0000 C CNN
 F 2 "" H 6500 3900 50  0000 C CNN
@@
 	6500 3900 6500 4050
 $Comp
-L GND #PWR07
+L GND #PWR110
 U 1 1 56AEF5AD
 P 6400 3900
-F 0 "#PWR07" H 6400 3650 50  0001 C CNN
+F 0 "#PWR110" H 6400 3650 50  0001 C CNN
 F 1 "GND" H 6400 3750 50  0000 C CNN
 F 2 "" H 6400 3900 50  0000 C CNN
@@
 	6400 3900 6400 4050
 $Comp
-L GND #PWR08
+L GND #PWR108
 U 1 1 56AEF5EA
 P 6200 3900
-F 0 "#PWR08" H 6200 3650 50  0001 C CNN
+F 0 "#PWR108" H 6200 3650 50  0001 C CNN
 F 1 "GND" H 6200 3750 50  0000 C CNN
 F 2 "" H 6200 3900 50  0000 C CNN
@@
 	6200 3900 6200 4050
 $Comp
-L GND #PWR09
+L GND #PWR115
 U 1 1 56AEF628
 P 7100 4550
-F 0 "#PWR09" H 7100 4300 50  0001 C CNN
+F 0 "#PWR115" H 7100 4300 50  0001 C CNN
 F 1 "GND" H 7100 4400 50  0000 C CNN
 F 2 "" H 7100 4550 50  0000 C CNN
@@
 	7000 4550 7100 4550
 $Comp
-L GND #PWR010
+L GND #PWR116
 U 1 1 56AEF667
 P 7100 4750
-F 0 "#PWR010" H 7100 4500 50  0001 C CNN
+F 0 "#PWR116" H 7100 4500 50  0001 C CNN
 F 1 "GND" H 7100 4600 50  0000 C CNN
 F 2 "" H 7100 4750 50  0000 C CNN
@@
 	7100 4750 7000 4750
 $Comp
-L GND #PWR011
+L GND #PWR117
 U 1 1 56AEF6A7
 P 7100 4850
-F 0 "#PWR011" H 7100 4600 50  0001 C CNN
+F 0 "#PWR117" H 7100 4600 50  0001 C CNN
 F 1 "GND" H 7100 4700 50  0000 C CNN
 F 2 "" H 7100 4850 50  0000 C CNN
@@
 	7100 4850 7000 4850
 $Comp
-L GND #PWR012
+L GND #PWR106
 U 1 1 56AEF70C
 P 5600 4550
-F 0 "#PWR012" H 5600 4300 50  0001 C CNN
+F 0 "#PWR106" H 5600 4300 50  0001 C CNN
 F 1 "GND" H 5600 4400 50  0000 C CNN
 F 2 "" H 5600 4550 50  0000 C CNN
@@
 	5600 4550 5700 4550
 $Comp
-L GND #PWR013
+L GND #PWR107
 U 1 1 56AEF771
 P 5600 4750
-F 0 "#PWR013" H 5600 4500 50  0001 C CNN
+F 0 "#PWR107" H 5600 4500 50  0001 C CNN
 F 1 "GND" H 5600 4600 50  0000 C CNN
 F 2 "" H 5600 4750 50  0000 C CNN
@@
 	0    -1   1    0
 $EndComp
-$Comp
-L CONN_SMA U1
-U 1 1 56AF18A3
-P 2600 3350
-F 0 "U1" H 2250 3550 60  0000 C CNN
-F 1 "CONN_SMA" H 2450 3700 60  0000 C CNN
-F 2 "vna_footprints:732511150_sma" H 2600 3350 60  0001 C CNN
-F 3 "" H 2600 3350 60  0000 C CNN
-	1    2600 3350
-	-1   0    0    -1
-$EndComp
-$Comp
-L GND #PWR014
-U 1 1 56AF18A9
-P 2600 4050
-F 0 "#PWR014" H 2600 3800 50  0001 C CNN
-F 1 "GND" H 2600 3900 50  0000 C CNN
-F 2 "" H 2600 4050 50  0000 C CNN
-F 3 "" H 2600 4050 50  0000 C CNN
-	1    2600 4050
-	-1   0    0    -1
-$EndComp
-Wire Wire Line
-	2750 3800 2750 3950
-Wire Wire Line
-	2750 3950 2450 3950
-Wire Wire Line
-	2450 3950 2450 3800
-Wire Wire Line
-	2550 3800 2550 3950
-Connection ~ 2550 3950
-Wire Wire Line
-	2650 3800 2650 3950
-Connection ~ 2650 3950
-Wire Wire Line
-	2600 3950 2600 4050
-Connection ~ 2600 3950
 Wire Wire Line
 	3350 3350 3150 3350
@@
 	5700 4850 4400 4850
 $Comp
-L GND #PWR015
+L GND #PWR103
 U 1 1 56AF1A38
 P 4550 4750
-F 0 "#PWR015" H 4550 4500 50  0001 C CNN
+F 0 "#PWR103" H 4550 4500 50  0001 C CNN
 F 1 "GND" H 4550 4600 50  0000 C CNN
 F 2 "" H 4550 4750 50  0000 C CNN
@@
 $EndComp
 $Comp
-L GND #PWR016
+L GND #PWR104
 U 1 1 56AF1B84
 P 4650 5300
-F 0 "#PWR016" H 4650 5050 50  0001 C CNN
+F 0 "#PWR104" H 4650 5050 50  0001 C CNN
 F 1 "GND" H 4650 5150 50  0000 C CNN
 F 2 "" H 4650 5300 50  0000 C CNN
@@
 Connection ~ 4650 4850
 $Comp
-L GND #PWR017
+L GND #PWR105
 U 1 1 56AF1C5F
 P 5000 5300
-F 0 "#PWR017" H 5000 5050 50  0001 C CNN
+F 0 "#PWR105" H 5000 5050 50  0001 C CNN
 F 1 "GND" H 5000 5150 50  0000 C CNN
 F 2 "" H 5000 5300 50  0000 C CNN
@@
 Connection ~ 5000 4850
 $Comp
-L mounting_box U5
-U 1 1 56B63F52
-P 6250 2550
-F 0 "U5" H 6250 2550 60  0000 C CNN
-F 1 "mounting_box" H 6200 2700 60  0000 C CNN
-F 2 "vna_footprints:POMONA_2400BOX" H 6250 2550 60  0001 C CNN
-F 3 "" H 6250 2550 60  0000 C CNN
-	1    6250 2550
-	1    0    0    -1
-$EndComp
-$Comp
-L GND #PWR018
+L GND #PWR114
 U 1 1 56CE6531
 P 7100 4450
-F 0 "#PWR018" H 7100 4200 50  0001 C CNN
+F 0 "#PWR114" H 7100 4200 50  0001 C CNN
 F 1 "GND" H 7100 4300 50  0000 C CNN
 F 2 "" H 7100 4450 50  0000 C CNN
@@
 Wire Wire Line
 	7100 4450 7000 4450
+$Comp
+L CONN_SMA_2GND U101
+U 1 1 576CF551
+P 2750 3350
+F 0 "U101" H 2450 3550 60  0000 C CNN
+F 1 "CONN_SMA_2GND" H 2800 3650 60  0000 C CNN
+F 2 "vna_footprints:142-0721-882_sma_cutout" H 2750 3350 60  0001 C CNN
+F 3 "" H 2750 3350 60  0000 C CNN
+	1    2750 3350
+	1    0    0    -1
+$EndComp
+$Comp
+L GND #PWR101
+U 1 1 576CF63E
+P 2750 3900
+F 0 "#PWR101" H 2750 3650 50  0001 C CNN
+F 1 "GND" H 2750 3750 50  0000 C CNN
+F 2 "" H 2750 3900 50  0000 C CNN
+F 3 "" H 2750 3900 50  0000 C CNN
+	1    2750 3900
+	-1   0    0    -1
+$EndComp
+Wire Wire Line
+	2750 3900 2750 3850
+Wire Wire Line
+	2700 3850 2800 3850
+Wire Wire Line
+	2700 3850 2700 3800
+Wire Wire Line
+	2800 3850 2800 3800
+Connection ~ 2750 3850
+$Comp
+L CONN_SMA_2GND U102
+U 1 1 576CF7C8
+P 2750 5750
+F 0 "U102" H 2450 5950 60  0000 C CNN
+F 1 "CONN_SMA_2GND" H 2800 6050 60  0000 C CNN
+F 2 "vna_footprints:142-0721-882_sma_cutout" H 2750 5750 60  0001 C CNN
+F 3 "" H 2750 5750 60  0000 C CNN
+	1    2750 5750
+	1    0    0    -1
+$EndComp
+$Comp
+L GND #PWR102
+U 1 1 576CF7CE
+P 2750 6300
+F 0 "#PWR102" H 2750 6050 50  0001 C CNN
+F 1 "GND" H 2750 6150 50  0000 C CNN
+F 2 "" H 2750 6300 50  0000 C CNN
+F 3 "" H 2750 6300 50  0000 C CNN
+	1    2750 6300
+	-1   0    0    -1
+$EndComp
+Wire Wire Line
+	2750 6300 2750 6250
+Wire Wire Line
+	2700 6250 2800 6250
+Wire Wire Line
+	2700 6250 2700 6200
+Wire Wire Line
+	2800 6250 2800 6200
+Connection ~ 2750 6250
+$Comp
+L CONN_SMA_2GND U103
+U 1 1 576CF92B
+P 9150 4650
+F 0 "U103" H 8850 4850 60  0000 C CNN
+F 1 "CONN_SMA_2GND" H 9200 4950 60  0000 C CNN
+F 2 "vna_footprints:142-0721-882_sma_cutout" H 9150 4650 60  0001 C CNN
+F 3 "" H 9150 4650 60  0000 C CNN
+	1    9150 4650
+	-1   0    0    -1
+$EndComp
+$Comp
+L GND #PWR118
+U 1 1 576CF931
+P 9150 5200
+F 0 "#PWR118" H 9150 4950 50  0001 C CNN
+F 1 "GND" H 9150 5050 50  0000 C CNN
+F 2 "" H 9150 5200 50  0000 C CNN
+F 3 "" H 9150 5200 50  0000 C CNN
+	1    9150 5200
+	1    0    0    -1
+$EndComp
+Wire Wire Line
+	9200 5150 9100 5150
+Wire Wire Line
+	9200 5150 9200 5100
+Wire Wire Line
+	9100 5150 9100 5100
+Wire Wire Line
+	9150 5200 9150 5150
+Connection ~ 9150 5150
 $EndSCHEMATC
