File: breakouts/amp_macom/amp_macom.sch (KiCad schematic (older format))
At the start: 8 parts, among them P1 CONN_01X02, U1 CONN_SMA, U2 CMM0511-QT-0G0T, U3 CONN_SMA

Commit message: work on ad9864 schematic, vco and if
Parts:
- U1, U3: footprint vna_footprints:732511150_sma_thin -> vna_footprints:SMA_CPW_1MM_.2MM
Changed lines of the file:
@@
 LIBS:txco
 LIBS:cmm0511-qt-0g0t
+LIBS:amp_macom-cache
 EELAYER 25 0
 EELAYER END
@@
 F 0 "U1" H 2350 4400 60  0000 C CNN
 F 1 "CONN_SMA" H 2550 4550 60  0000 C CNN
-F 2 "vna_footprints:732511150_sma_thin" H 2700 4200 60  0001 C CNN
+F 2 "vna_footprints:SMA_CPW_1MM_.2MM" H 2700 4200 60  0001 C CNN
 F 3 "" H 2700 4200 60  0000 C CNN
 	1    2700 4200
@@
 F 0 "U3" H 7850 4400 60  0000 C CNN
 F 1 "CONN_SMA" H 8050 4550 60  0000 C CNN
-F 2 "vna_footprints:732511150_sma_thin" H 8200 4200 60  0001 C CNN
+F 2 "vna_footprints:SMA_CPW_1MM_.2MM" H 8200 4200 60  0001 C CNN
 F 3 "" H 8200 4200 60  0000 C CNN
 	1    8200 4200
