File: hardware/mm_reflectometer/evalboards/ecp5/bias.kicad_sch (KiCad schematic)
At the start: 35 parts, among them J601 Conn_Coaxial, J602 Conn_Coaxial, U101 ECP5U_25_CABGA256, U603 ADS7868, U604 DAC7563SDSCR, U605 OPA2140, U606 TS5A23166

Commit message: routing on ecp5 eval board
Parts:
- removed R611, R612: 10k, Resistor_SMD:R_0402_1005Metric, symbol Device:R_Small
Connections:
- net SDA is gone; now on net SYNTH_VT_CS: U101.A15 (PT67B/-)
- net ADC_SCK: now also U101.A14 (PT65B/-); no longer U101.B13 (PT60A/+)
- net ADC_SDO: now also U101.A13 (PT65A/+); no longer U101.E12 (PT58B/-)
- net DAC_DIN: now also U101.A12 (PT53B/-); no longer U101.E11 (PT51B/-)
- net DAC_SCLK: now also U101.A10 (PT42B/-); no longer U101.D11 (PT51A/+)
- net DAC_~SYNC: now also U101.B10 (PT44A/+); no longer U101.C11 (PT49B/-)
- net M5V_EN: now also U101.B12 (PT56A/+); no longer U101.C12 (PT56B/-)
- net SYNTH_VT_CS: no longer U101.C13 (PT60B/-)
- net at U101.B8 (PT35B/-/PCLKC1_0): now also J601.1 (In)
- net at U101.C8 (PT35A/+/PCLKT1_0): now also J602.1 (In)
- net at U101.D8 (PT33B/-/PCLKC1_1): no longer J602.1 (In)
- net at U101.E8 (PT33A/+/PCLKT1_1): no longer J601.1 (In)
- net SCL: no longer names the net of U101.B14 (PT67A/+)
Other:
- moved on the sheet: J601, J602

Commit message: cleanup ecp5 schematic, generated assembly drawings
Parts:
- R605, R606: value 33k -> 4.7k
- R607, R608: value 10k -> 33k
Changed lines of the file:
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@@
   (junction (at 335.28 27.94) (diameter 0.9144) (color 0 0 0 0))
   (junction (at 345.44 27.94) (diameter 0.9144) (color 0 0 0 0))
+  (no_connect (at 321.31 54.61))
   (no_connect (at 349.25 54.61))
-  (no_connect (at 321.31 54.61))
   (wire (pts (xy 13.97 39.37) (xy 26.67 39.37))
     (stroke (width 0) (type solid) (color 0 0 0 0))
@@
     (in_bom yes) (on_board yes)
     (property "Reference" "R605" (id 0) (at 252.73 153.7716 90))
-    (property "Value" "33k" (id 1) (at 252.73 156.083 90))
+    (property "Value" "4.7k" (id 1) (at 252.73 156.083 90))
     (property "Footprint" "Resistor_SMD:R_0402_1005Metric" (id 2) (at 252.73 158.75 0)
       (effects (font (size 1.27 1.27)) hide)
@@
     (in_bom yes) (on_board yes)
     (property "Reference" "R606" (id 0) (at 252.73 171.5516 90))
-    (property "Value" "33k" (id 1) (at 252.73 173.863 90))
+    (property "Value" "4.7k" (id 1) (at 252.73 173.863 90))
     (property "Footprint" "Resistor_SMD:R_0402_1005Metric" (id 2) (at 252.73 176.53 0)
       (effects (font (size 1.27 1.27)) hide)
@@
     (in_bom yes) (on_board yes)
     (property "Reference" "R607" (id 0) (at 264.0584 186.69 90))
-    (property "Value" "10k" (id 1) (at 261.747 186.69 90))
+    (property "Value" "33k" (id 1) (at 261.747 186.69 90))
     (property "Footprint" "Resistor_SMD:R_0402_1005Metric" (id 2) (at 259.08 186.69 0)
       (effects (font (size 1.27 1.27)) hide)
@@
     (in_bom yes) (on_board yes)
     (property "Reference" "R608" (id 0) (at 270.51 153.7716 90))
-    (property "Value" "10k" (id 1) (at 270.51 156.083 90))
+    (property "Value" "33k" (id 1) (at 270.51 156.083 90))
     (property "Footprint" "Resistor_SMD:R_0402_1005Metric" (id 2) (at 270.51 158.75 0)
       (effects (font (size 1.27 1.27)) hide)
