File: hardware/mm_reflectometer/evalboards/mamx_011036/mamx_011036.kicad_pcb (KiCad board)
At the start: 4 copper layers, 28.1 x 31.4 mm, 37 parts, among them J1 Screw_Terminal_01x02, J2 Conn_Coaxial, J3 Conn_Coaxial, J4 Conn_Coaxial, Q1 IRLML6401, Q2 BC848W, Q3 IRLML6401, U1 LM27761, U2 ADM7170ACPZ-5.0-R7, U3 MAAM-011109, U4 MAMX-011036

Commit message: cleanup ecp5 schematic, generated assembly drawings
Parts:
- R2: value 10k -> 158k
- R3: value 10k -> 51k
Connections:
- U3 pad 3: no_connect_25 -> (no net)
- U3 pad 4: no_connect_26 -> (no net)
- U3 pad 7: no_connect_27 -> (no net)
- U3 pad 9: no_connect_28 -> (no net)
Changed lines of the file:
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@@
   (net 22 "Net-(R2-Pad2)")
   (net 23 "Net-(TP6-Pad1)")
-  (net 24 "no_connect_28")
-  (net 25 "no_connect_27")
-  (net 26 "Net-(U3-Pad5)")
-  (net 27 "no_connect_26")
-  (net 28 "no_connect_25")
+  (net 24 "Net-(U3-Pad5)")
   (footprint "jtk_rf_footprints:sw_edge_oshpark_4layer" (layer "F.Cu")
     (at 115 78.550001 180)
@@
       (effects (font (size 0.7 0.7) (thickness 0.15)))
     )
-    (fp_text value "10k" (at 0 1.17 90) (layer "F.Fab")
+    (fp_text value "51k" (at 0 1.17 90) (layer "F.Fab")
       (effects (font (size 1 1) (thickness 0.15)))
     )
@@
       (net 1 "GND") (pinfunction "GND"))
     (pad "2" smd roundrect (at -1.2475 0) (size 0.4 0.3) (layers "F.Cu" "F.Paste" "F.Mask") (roundrect_rratio 0.25)
-      (net 26 "Net-(U3-Pad5)") (pinfunction "LO"))
+      (net 24 "Net-(U3-Pad5)") (pinfunction "LO"))
     (pad "3" smd roundrect (at -1.2475 0.5) (size 0.4 0.3) (layers "F.Cu" "F.Paste" "F.Mask") (roundrect_rratio 0.25)
       (net 1 "GND") (pinfunction "GND"))
@@
       (net 9 "-5V") (pinfunction "Ve"))
     (pad "3" smd roundrect (at 0 2.075 90) (size 0.65 0.4) (layers "F.Cu" "F.Paste" "F.Mask") (roundrect_rratio 0.25)
-      (net 28 "no_connect_25") (pinfunction "NC"))
+      (pinfunction "NC"))
     (pad "4" smd roundrect (at 0.7 2.075 90) (size 0.65 0.4) (layers "F.Cu" "F.Paste" "F.Mask") (roundrect_rratio 0.25)
-      (net 27 "no_connect_26") (pinfunction "Vg"))
+      (pinfunction "Vg"))
     (pad "5" smd roundrect (at 2.075 0) (size 0.65 0.4) (layers "F.Cu" "F.Paste" "F.Mask") (roundrect_rratio 0.25)
-      (net 26 "Net-(U3-Pad5)") (pinfunction "RFout"))
+      (net 24 "Net-(U3-Pad5)") (pinfunction "RFout"))
     (pad "6" smd roundrect (at 0.7 -2.075 90) (size 0.65 0.4) (layers "F.Cu" "F.Paste" "F.Mask") (roundrect_rratio 0.25)
       (net 16 "Net-(L1-Pad2)") (pinfunction "Vd"))
     (pad "7" smd roundrect (at 0 -2.075 90) (size 0.65 0.4) (layers "F.Cu" "F.Paste" "F.Mask") (roundrect_rratio 0.25)
-      (net 25 "no_connect_27") (pinfunction "Bc"))
+      (pinfunction "Bc"))
     (pad "8" smd roundrect (at -0.7 -2.075 90) (size 0.65 0.4) (layers "F.Cu" "F.Paste" "F.Mask") (roundrect_rratio 0.25)
       (net 23 "Net-(TP6-Pad1)") (pinfunction "Vdet"))
     (pad "9" smd roundrect (at -1.4 -2.075 90) (size 0.65 0.4) (layers "F.Cu" "F.Paste" "F.Mask") (roundrect_rratio 0.25)
-      (net 24 "no_connect_28") (pinfunction "Vc"))
+      (pinfunction "Vc"))
     (pad "10" smd rect (at 1.85 -2 90) (size 1 1.3) (layers "F.Cu" "F.Paste" "F.Mask")
       (net 1 "GND") (pinfunction "EP") (solder_paste_margin -0.15))
@@
       (effects (font (size 0.7 0.7) (thickness 0.15)))
     )
-    (fp_text value "10k" (at 0 1.17 90) (layer "F.Fab")
+    (fp_text value "158k" (at 0 1.17 90) (layer "F.Fab")
       (effects (font (size 1 1) (thickness 0.15)))
     )
@@
   (segment (start 109 65) (end 108.5 65) (width 0.25) (layer "F.Cu") (net 23))
   (segment (start 109.3 65.3) (end 109 65) (width 0.25) (layer "F.Cu") (net 23))
-  (segment (start 113 68.5) (end 113.344606 68.5) (width 0.39) (layer "F.Cu") (net 26))
-  (segment (start 112.075 68.5) (end 113 68.5) (width 0.39) (layer "F.Cu") (net 26))
+  (segment (start 113 68.5) (end 113.344606 68.5) (width 0.39) (layer "F.Cu") (net 24))
+  (segment (start 112.075 68.5) (end 113 68.5) (width 0.39) (layer "F.Cu") (net 24))
   (zone (net 1) (net_name "GND") (layer "F.Cu") (hatch edge 0.508)
     (priority 2)
@@
     )
   )
-  (zone (net 26) (net_name "Net-(U3-Pad5)") (layer "F.Cu") (hatch edge 0.508)
+  (zone (net 24) (net_name "Net-(U3-Pad5)") (layer "F.Cu") (hatch edge 0.508)
     (connect_pads yes (clearance 0.127))
     (min_thickness 0.127) (filled_areas_thickness no)
