File: hardware/mm_reflectometer/evalboards/xx1000-qt/mmic_bias.kicad_sch (KiCad schematic)
At the start: 22 parts, among them U5 TLV9151IDCKR

Commit message: schematic work on mm synth -- starting voltage regulation
Parts:
- R13: value DNI -> 0
- R15: value 0.5 -> 0
- R19: value 0 -> DNI
Changed lines of the file:
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@@
-(kicad_sch (version 20210126) (generator eeschema)
+(kicad_sch (version 20210406) (generator eeschema)
   (paper "A4")
   (junction (at 184.15 93.98) (diameter 1.016) (color 0 0 0 0))
@@
   (symbol (lib_id "power:+5V") (at 212.09 74.93 90) (unit 1)
     (in_bom yes) (on_board yes)
-    (property "Reference" "#PWR?" (id 0) (at 215.9 74.93 0)
+    (property "Reference" "#PWR0134" (id 0) (at 215.9 74.93 0)
       (effects (font (size 1.27 1.27)) hide)
     )
@@
   (symbol (lib_id "power:+5V") (at 262.89 35.56 0) (unit 1)
     (in_bom yes) (on_board yes)
-    (property "Reference" "#PWR?" (id 0) (at 262.89 39.37 0)
+    (property "Reference" "#PWR0135" (id 0) (at 262.89 39.37 0)
       (effects (font (size 1.27 1.27)) hide)
     )
@@
     (in_bom yes) (on_board yes)
     (property "Reference" "R13" (id 0) (at 208.28 97.79 0))
-    (property "Value" "DNI" (id 1) (at 208.28 100.33 0))
+    (property "Value" "0" (id 1) (at 208.28 100.33 0))
     (property "Footprint" "Resistor_SMD:R_0402_1005Metric" (id 2) (at 210.82 99.06 0)
       (effects (font (size 1.27 1.27)) hide)
@@
       (effects (font (size 1.27 1.27)) (justify left))
     )
-    (property "Value" "0.5" (id 1) (at 214.63 52.07 0)
+    (property "Value" "0" (id 1) (at 214.63 52.07 0)
       (effects (font (size 1.27 1.27)) (justify left))
     )
@@
     (in_bom yes) (on_board yes)
     (property "Reference" "R19" (id 0) (at 214.63 96.52 0))
-    (property "Value" "0" (id 1) (at 217.17 96.52 0))
+    (property "Value" "DNI" (id 1) (at 217.17 96.52 0))
     (property "Footprint" "Resistor_SMD:R_0402_1005Metric" (id 2) (at 215.9 93.98 0)
       (effects (font (size 1.27 1.27)) hide)
