File: hardware/mm_reflectometer/evalboards/xx1000-qt/xx1000-qt.kicad_pcb (KiCad board)
At the start: 4 copper layers, 28.1 x 33.6 mm, 60 parts, among them J1 Screw_Terminal_01x02, J3 Conn_Coaxial, J4 Conn_Coaxial, Q1 IRLML6401, Q2 BC848W, Q3 IRLML6401, U1 LM27761, U2 ADM7170ACPZ-5.0-R7, U3 XX1000-QT, U5 TLV9151IDCKR

Commit message: schematic work on mm synth -- starting voltage regulation
Parts:
- R13: value DNI -> 0
- R15: value 0.5 -> 0
- R19: value 0 -> DNI
