File: hardware/mm_reflectometer/synth/mm_synth/refclk.kicad_sch (KiCad schematic)
At the start: 116 parts

Commit message: added dac to mm_synth for vtune/adjstable bias, added ADC for telemetry
Parts:
- removed C? (x7): 2.2 uF, Capacitor_SMD:C_0603_1608Metric, symbol Device:C_Small
- removed C? (x12): 10 nF, Capacitor_SMD:C_0402_1005Metric, symbol Device:C_Small
- removed C?: 220 nF, Capacitor_SMD:C_0402_1005Metric, symbol Device:C_Small
- removed C? (x2): 0.0033uF, Capacitor_SMD:C_0402_1005Metric, symbol Device:C_Small
- removed C? (x9): 100 nF, Capacitor_SMD:C_0402_1005Metric, symbol Device:C_Small
- removed C?: 47 pF, Capacitor_SMD:C_0402_1005Metric, symbol Device:C_Small
- removed C?: 15 pF, Capacitor_SMD:C_0402_1005Metric, symbol Device:C_Small
- removed C? (x7): 100 pF, Capacitor_SMD:C_0402_1005Metric, symbol Device:C_Small
- removed C?: 4.5 pF, Capacitor_SMD:C_0402_1005Metric, symbol Device:C_Small
- removed C? (x3): DNI, Capacitor_SMD:C_0402_1005Metric, symbol Device:C_Small
- removed C?: 2.2 nF, Capacitor_SMD:C_0402_1005Metric, symbol Device:C_Small
- removed C?: 22 uF, Capacitor_SMD:C_0805_2012Metric, symbol Device:C_Small
- removed C?: 4.7 uF, Capacitor_SMD:C_0603_1608Metric, symbol Device:C_Small
- removed C? (x2): JMP, Capacitor_SMD:C_0402_1005Metric, symbol Device:C_Small
- removed C?: 220 pF, Capacitor_SMD:C_0402_1005Metric, symbol Device:C_Small
- removed D?: RED, LED_SMD:LED_0603_1608Metric, symbol Device:LED_Small
- removed D? (x3): TPD1E04U04, Diode_SMD:D_0402_1005Metric, symbol Device:D_TVS
- removed D?: CGRTS4001-HF, Diode_SMD:D_SOD-123F, symbol Device:D_Small
- removed J? (x4): SMA, Connector_Coaxial:SMA_Amphenol_132289_EdgeMount, symbol Connector:Conn_Coaxial
- removed K?: 1-1462051-1, Relay_SMD:Relay_SPDT_AXICOM_HF3Series_50ohms_Pitch1.27mm, symbol vna_mm_ref-rescue:1-1462051-1-vna_mm
- removed L?: BLM18EG101TN1D, Inductor_SMD:L_0603_1608Metric, symbol Device:L_Small
- removed L? (x6): BLM15AG102SZ1D, Inductor_SMD:L_0402_1005Metric, symbol Device:L_Small
- removed L?: JMP, Inductor_SMD:L_0805_2012Metric, symbol Device:L_Small
- removed L?: DNI, Inductor_SMD:L_0402_1005Metric, symbol Device:L_Small
- removed L?: 11 nH, Inductor_SMD:L_0402_1005Metric, symbol Device:L_Small
- removed L?: 560 nH, Inductor_SMD:L_0805_2012Metric, symbol Device:L_Small
- removed L?: 110 nH, Inductor_SMD:L_0603_1608Metric, symbol Device:L_Small
- removed L?: 5.6 uH, Inductor_SMD:L_0805_2012Metric, symbol Device:L_Small
- removed R? (x7): 10k, Resistor_SMD:R_0402_1005Metric, symbol Device:R_Small
- removed R? (x6): DNI, Resistor_SMD:R_0402_1005Metric, symbol Device:R_Small
- removed R? (x2): 50, Resistor_SMD:R_0402_1005Metric, symbol Device:R_Small
- removed R? (x4): 51, Resistor_SMD:R_0402_1005Metric, symbol Device:R_Small
- removed R? (x4): 0, Resistor_SMD:R_0402_1005Metric, symbol Device:R_Small
- removed R? (x4): 75, Resistor_SMD:R_0402_1005Metric, symbol Device:R_Small
- removed R?: JMP, Resistor_SMD:R_0402_1005Metric, symbol Device:R_Small
- removed R? (x4): 100, Resistor_SMD:R_0402_1005Metric, symbol Device:R_Small
- removed R?: 7.5k, Resistor_SMD:R_0402_1005Metric, symbol Device:R_Small
- removed TP?: V_RELAY, TestPoint:TestPoint_Keystone_5015_Micro-Minature, symbol Connector:TestPoint
- removed TP?: VCTRL, TestPoint:TestPoint_Keystone_5015_Micro-Minature, symbol Connector:TestPoint
- removed TP?: CP, TestPoint:TestPoint_Keystone_5015_Micro-Minature, symbol Connector:TestPoint
- removed U? (x2): LTC6957xDD-3, Package_DFN_QFN:DFN-12-1EP_3x3mm_P0.45mm_EP1.66x2.38mm, symbol Interface:LTC6957xDD-3
- removed U?: HMC1031, Package_SO:MSOP-8_3x3mm_P0.65mm, symbol vna_mm_ref-rescue:HMC1031-vna_mm
- removed U?: 74AHC1G04, Package_TO_SOT_SMD:SOT-353_SC-70-5, symbol 74xGxx:74AHC1G04
- removed U?: DOCAT050F-010.0M, vna_mm:DOCAT_9.1x14.1mm, symbol vna_mm_ref-rescue:DOCAT-vna_mm
- removed U?: DRV8837C, Package_SON:WSON-8-1EP_2x2mm_P0.5mm_EP0.9x1.6mm, symbol Driver_Motor:DRV8837C
- removed X?: ABLNO-V-100.000MHZ, Oscillator:Oscillator_SMD_Abracon_ABLNO, symbol Oscillator:ABLNO
- added C?: 22 uF, Capacitor_SMD:C_0805_2012Metric, symbol Device:C_Small
- added C? (x4): 100 nF, Capacitor_SMD:C_0402_1005Metric, symbol Device:C_Small
- added C?: 47 pF, Capacitor_SMD:C_0402_1005Metric, symbol Device:C_Small
- added C?: 100 pF, Capacitor_SMD:C_0402_1005Metric, symbol Device:C_Small
- added C?: JMP, Capacitor_SMD:C_0402_1005Metric, symbol Device:C_Small
- added C?: 2.2 uF, Capacitor_SMD:C_0603_1608Metric, symbol Device:C_Small
- added C?: 2.2 nF, Capacitor_SMD:C_0402_1005Metric, symbol Device:C_Small
- added D?: CGRTS4001-HF, Diode_SMD:D_SOD-123F, symbol Device:D_Small
- added D?: TPD1E04U04, Diode_SMD:D_0402_1005Metric, symbol Device:D_TVS
- added K?: 1-1462051-1, Relay_SMD:Relay_SPDT_AXICOM_HF3Series_50ohms_Pitch1.27mm, symbol vna_mm_ref-rescue:1-1462051-1-vna_mm
- added L?: BLM15AG102SZ1D, Inductor_SMD:L_0402_1005Metric, symbol Device:L_Small
- added L?: 110 nH, Inductor_SMD:L_0603_1608Metric, symbol Device:L_Small
- added L?: 5.6 uH, Inductor_SMD:L_0805_2012Metric, symbol Device:L_Small
- added Q?: IRLML6401, Package_TO_SOT_SMD:SOT-23, symbol Transistor_FET:IRLML6401
- added R?: 10k, Resistor_SMD:R_0402_1005Metric, symbol Device:R_Small
- added R?: 1k, Resistor_SMD:R_0402_1005Metric, symbol Device:R_Small
- added R?: 22, Resistor_SMD:R_0402_1005Metric, symbol Device:R_Small
- added R? (x2): DNI, Resistor_SMD:R_0402_1005Metric, symbol Device:R_Small
- added R?: JMP, Resistor_SMD:R_0402_1005Metric, symbol Device:R_Small
- added U?: DRV8837C, Package_SON:WSON-8-1EP_2x2mm_P0.5mm_EP0.9x1.6mm, symbol Driver_Motor:DRV8837C
- added U?: 74AHC1G04, Package_TO_SOT_SMD:SOT-353_SC-70-5, symbol 74xGxx:74AHC1G04
- added X?: ABLNO-100.000MHZ, Oscillator:Oscillator_SMD_Abracon_ABLNO, symbol Oscillator:ABLNO
Connections:
- net +3V3: now also Q?.2 (S), R?.2
- net +4V: now also C?.1, D?.2 (A), U?.5 (VCC), U?.8 (VCC)
- net GND: now also C?.1, C?.2, C?.2, C?.2, C?.2, C?.2, C?.2, C?.2, D?.2 (A2), K?.10, K?.13, K?.15, K?.17, K?.19, K?.2, K?.21, K?.5, K?.7, L?.1, R?.1, U?.3 (GND), U?.4 (GND), U?.9 (GND), X?.2 (GND)
- net REF_SEL: now also U?.2, U?.6 (IN1)
- net RELAY_EN: now also U?.7 (~SLEEP)
- new net: L?.1, Q?.3 (D)
- new net: C?.1, C?.1, C?.1, L?.2, X?.4 (VDD)
- new net: C?.1, C?.1, D?.1 (K), U?.1 (VM)
- new net: C?.1, Q?.1 (G), R?.1, R?.1
- new net: K?.11, K?.22 (S), U?.2 (OUT1)
- new net: K?.1, K?.12 (R), U?.3 (OUT2)
- new net: U?.4, U?.5 (IN2)
- new net: K?.14, R?.1
- new net: R?.2, X?.3 (RFout)
- new net: C?.1, L?.2
- new net: C?.2, C?.2, L?.2, R?.1, R?.2
- new net: D?.1 (A1), K?.20, L?.1, R?.2
- new net: C?.1, R?.2
- new net OSC_OUT: K?.6, R?.1
- new net REF_EN: R?.2
- new net REF_IN: C?.2
- no-connect marks 0 -> 1
Other:
- note added: "0.3 to 3.6Vpp into LMX2820, AC coupled, 50 ohm input impedance"
- note removed: "2 mA typical"
- note removed: "30 mA"
- note removed: "3Vpp"
- note removed: "5 mA"
- note removed: "HMC1031 recommended input region is 0.2 to 3.3 Vpp"
- note removed: "MATCH INPUT IMPEDANCE 3600 OHM ||4 pF"
- note removed: "TODO: TPD1E04U04 IS A BAD CHOICE FOR AC COUPLED SIGNALS, WILL CLIP BELOW 0.7V. FIND A NEW TVS DIODE"
- note removed: "Target 0.5 Vpp"
- note removed: "USE LOW LEAKAGE MLCC CAPS"
- note removed: "VCOIN input region is 0.2 to 1.5 Vpp"

Commit message: started digital control schematic page on mm_synth, removed stale documentation
Parts:
- R?: value 22 -> 33
Other:
- note added: "TODO: CHANGE RELAY DRIVER VOLTAGE"
Changed lines of the file:
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@@
     (effects (font (size 1.27 1.27)) (justify left bottom))
+  )
+  (text "TODO: CHANGE RELAY DRIVER VOLTAGE" (at 190.5 22.86 180)
+    (effects (font (size 3 3)) (justify right bottom))
   )
   (text "0.3 to 3.6Vpp into LMX2820, AC coupled, 50 ohm input impedance\n"
@@
       (effects (font (size 1.27 1.27)) (justify right))
     )
-    (property "Value" "22" (id 1) (at 107.823 178.841 0)
-      (effects (font (size 1.27 1.27)) (justify right))
-    )
+    (property "Value" "33" (id 1) (at 107.823 178.841 0)
+      (effects (font (size 1.27 1.27)) (justify right))
+    )

Commit message: schematic work on mm synth -- starting voltage regulation
Parts:
- removed D?: CGRTS4001-HF, Diode_SMD:D_SOD-123F, symbol Device:D_Small
- D?: value TPD1E04U04 -> TPD1E1B04
- K?: value 1-1462051-1 -> 1-1462051-2
Connections:
- net +5VA: now reaches C?.1, C?.1, U?.1 (VM)
- net +5VA: now also C?.1, U?.8 (VCC)
- net +3V3 renamed +3.3VP
- removed net +4V: C?.1, U?.5 (VCC), U?.8 (VCC)
- new net +5VP: U?.5 (VCC)
Other:
- note added: "33 mA, bistable"
- note removed: "TODO: CHANGE RELAY DRIVER VOLTAGE"
Changed lines of the file:
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@@
-(kicad_sch (version 20210126) (generator eeschema)
+(kicad_sch (version 20210406) (generator eeschema)
   (paper "A4")
   (junction (at 45.72 146.05) (diameter 0.9144) (color 0 0 0 0))
@@
   (junction (at 114.3 110.49) (diameter 0.9144) (color 0 0 0 0))
   (junction (at 132.08 34.29) (diameter 0.9144) (color 0 0 0 0))
-  (junction (at 133.35 21.59) (diameter 0.9144) (color 0 0 0 0))
+  (junction (at 133.35 20.32) (diameter 0.9144) (color 0 0 0 0))
   (junction (at 134.62 34.29) (diameter 0.9144) (color 0 0 0 0))
   (junction (at 140.97 34.29) (diameter 0.9144) (color 0 0 0 0))
@@
     (stroke (width 0) (type solid) (color 0 0 0 0))
   )
-  (wire (pts (xy 45.72 144.78) (xy 45.72 146.05))
+  (wire (pts (xy 45.72 143.51) (xy 45.72 146.05))
     (stroke (width 0) (type solid) (color 0 0 0 0))
   )
@@
     (stroke (width 0) (type solid) (color 0 0 0 0))
   )
-  (wire (pts (xy 132.08 21.59) (xy 132.08 34.29))
+  (wire (pts (xy 132.08 20.32) (xy 132.08 34.29))
     (stroke (width 0) (type solid) (color 0 0 0 0))
   )
@@
     (stroke (width 0) (type solid) (color 0 0 0 0))
   )
-  (wire (pts (xy 133.35 21.59) (xy 132.08 21.59))
-    (stroke (width 0) (type solid) (color 0 0 0 0))
-  )
-  (wire (pts (xy 133.35 21.59) (xy 133.35 19.05))
-    (stroke (width 0) (type solid) (color 0 0 0 0))
-  )
-  (wire (pts (xy 134.62 21.59) (xy 133.35 21.59))
-    (stroke (width 0) (type solid) (color 0 0 0 0))
-  )
-  (wire (pts (xy 134.62 25.4) (xy 134.62 21.59))
-    (stroke (width 0) (type solid) (color 0 0 0 0))
-  )
-  (wire (pts (xy 134.62 30.48) (xy 134.62 34.29))
+  (wire (pts (xy 133.35 19.05) (xy 133.35 20.32))
+    (stroke (width 0) (type solid) (color 0 0 0 0))
+  )
+  (wire (pts (xy 133.35 20.32) (xy 132.08 20.32))
+    (stroke (width 0) (type solid) (color 0 0 0 0))
+  )
+  (wire (pts (xy 133.35 20.32) (xy 134.62 20.32))
+    (stroke (width 0) (type solid) (color 0 0 0 0))
+  )
+  (wire (pts (xy 134.62 20.32) (xy 134.62 34.29))
     (stroke (width 0) (type solid) (color 0 0 0 0))
   )
@@
     (effects (font (size 1.27 1.27)) (justify left bottom))
   )
-  (text "TODO: CHANGE RELAY DRIVER VOLTAGE" (at 190.5 22.86 180)
-    (effects (font (size 3 3)) (justify right bottom))
+  (text "33 mA, bistable" (at 138.43 53.975 0)
+    (effects (font (size 1.27 1.27)) (justify left bottom))
   )
   (text "0.3 to 3.6Vpp into LMX2820, AC coupled, 50 ohm input impedance\n"
@@
     (effects (font (size 1.27 1.27)) (justify left))
   )
+  (symbol (lib_id "power:+3.3VP") (at 45.72 143.51 0) (unit 1)
+    (in_bom yes) (on_board yes)
+    (property "Reference" "#PWR?" (id 0) (at 49.53 144.78 0)
+      (effects (font (size 1.27 1.27)) hide)
+    )
+    (property "Value" "+3.3VP" (id 1) (at 46.99 138.43 0))
+    (property "Footprint" "" (id 2) (at 45.72 143.51 0)
+      (effects (font (size 1.27 1.27)) hide)
+    )
+    (property "Datasheet" "" (id 3) (at 45.72 143.51 0)
+      (effects (font (size 1.27 1.27)) hide)
+    )
+    (pin "1")
+  )
+  (symbol (lib_id "power:+5VP") (at 99.06 72.39 0) (unit 1)
+    (in_bom yes) (on_board yes) (fields_autoplaced)
+    (property "Reference" "#PWR?" (id 0) (at 99.06 76.2 0)
+      (effects (font (size 1.27 1.27)) hide)
+    )
+    (property "Value" "+5VP" (id 1) (at 99.06 68.58 0))
+    (property "Footprint" "" (id 2) (at 99.06 72.39 0)
+      (effects (font (size 1.27 1.27)) hide)
+    )
+    (property "Datasheet" "" (id 3) (at 99.06 72.39 0)
+      (effects (font (size 1.27 1.27)) hide)
+    )
+    (pin "1")
+  )
+  (symbol (lib_id "power:+5VA") (at 133.35 19.05 0) (unit 1)
+    (in_bom yes) (on_board yes)
+    (property "Reference" "#PWR?" (id 0) (at 133.35 22.86 0)
+      (effects (font (size 1.27 1.27)) hide)
+    )
+    (property "Value" "+5VA" (id 1) (at 134.62 13.97 0))
+    (property "Footprint" "" (id 2) (at 133.35 19.05 0)
+      (effects (font (size 1.27 1.27)) hide)
+    )
+    (property "Datasheet" "" (id 3) (at 133.35 19.05 0)
+      (effects (font (size 1.27 1.27)) hide)
+    )
+    (pin "1")
+  )
   (symbol (lib_id "Device:L_Small") (at 77.47 118.11 0) (mirror x) (unit 1)
     (in_bom yes) (on_board yes)
@@
     (pin "1")
     (pin "2")
-  )
-  (symbol (lib_id "power:+3V3") (at 45.72 144.78 0) (unit 1)
-    (in_bom yes) (on_board yes)
-    (property "Reference" "#PWR?" (id 0) (at 45.72 148.59 0)
-      (effects (font (size 1.27 1.27)) hide)
-    )
-    (property "Value" "+3V3" (id 1) (at 46.101 140.3858 0))
-    (property "Footprint" "" (id 2) (at 45.72 144.78 0)
-      (effects (font (size 1.27 1.27)) hide)
-    )
-    (property "Datasheet" "" (id 3) (at 45.72 144.78 0)
-      (effects (font (size 1.27 1.27)) hide)
-    )
-    (pin "1")
-  )
-  (symbol (lib_id "power:+4V") (at 99.06 72.39 0) (unit 1)
-    (in_bom yes) (on_board yes)
-    (property "Reference" "#PWR?" (id 0) (at 99.06 76.2 0)
-      (effects (font (size 1.27 1.27)) hide)
-    )
-    (property "Value" "+4V" (id 1) (at 99.441 67.9958 0))
-    (property "Footprint" "" (id 2) (at 99.06 72.39 0)
-      (effects (font (size 1.27 1.27)) hide)
-    )
-    (property "Datasheet" "" (id 3) (at 99.06 72.39 0)
-      (effects (font (size 1.27 1.27)) hide)
-    )
-    (pin "1")
-  )
-  (symbol (lib_id "power:+4V") (at 133.35 19.05 0) (unit 1)
-    (in_bom yes) (on_board yes)
-    (property "Reference" "#PWR?" (id 0) (at 133.35 22.86 0)
-      (effects (font (size 1.27 1.27)) hide)
-    )
-    (property "Value" "+4V" (id 1) (at 133.731 14.6558 0))
-    (property "Footprint" "" (id 2) (at 133.35 19.05 0)
-      (effects (font (size 1.27 1.27)) hide)
-    )
-    (property "Datasheet" "" (id 3) (at 133.35 19.05 0)
-      (effects (font (size 1.27 1.27)) hide)
-    )
-    (pin "1")
   )
   (symbol (lib_id "power:GND") (at 45.72 173.99 0) (unit 1)
@@
     )
     (property "Datasheet" "~" (id 3) (at 173.99 134.62 0)
-      (effects (font (size 1.27 1.27)) hide)
-    )
-    (pin "1")
-    (pin "2")
-  )
-  (symbol (lib_id "Device:D_Small") (at 134.62 27.94 90) (unit 1)
-    (in_bom yes) (on_board yes)
-    (property "Reference" "D?" (id 0) (at 136.3472 26.7716 90)
-      (effects (font (size 1.27 1.27)) (justify right))
-    )
-    (property "Value" "CGRTS4001-HF" (id 1) (at 136.3472 29.083 90)
-      (effects (font (size 1.27 1.27)) (justify right))
-    )
-    (property "Footprint" "Diode_SMD:D_SOD-123F" (id 2) (at 134.62 27.94 90)
-      (effects (font (size 1.27 1.27)) hide)
-    )
-    (property "Datasheet" "~" (id 3) (at 134.62 27.94 90)
-      (effects (font (size 1.27 1.27)) hide)
-    )
-    (property "DIST_NAME" "Digi-Key" (id 4) (at 134.62 27.94 0)
-      (effects (font (size 1.27 1.27)) hide)
-    )
-    (property "DIST_PN" "641-2032-1-ND" (id 5) (at 134.62 27.94 0)
       (effects (font (size 1.27 1.27)) hide)
     )
@@
       (effects (font (size 1.27 1.27)) (justify left))
     )
-    (property "Value" "TPD1E04U04" (id 1) (at 116.3066 119.253 90)
+    (property "Value" "TPD1E1B04" (id 1) (at 116.3066 119.253 90)
       (effects (font (size 1.27 1.27)) (justify left))
     )
@@
     (in_bom yes) (on_board yes)
     (property "Reference" "K?" (id 0) (at 172.72 93.5482 0))
-    (property "Value" "1-1462051-1" (id 1) (at 172.72 95.8596 0))
+    (property "Value" "1-1462051-2" (id 1) (at 172.72 95.8596 0))
     (property "Footprint" "Relay_SMD:Relay_SPDT_AXICOM_HF3Series_50ohms_Pitch1.27mm" (id 2) (at 182.88 93.98 0)
       (effects (font (size 1.27 1.27)) (justify left) hide)
