File: hardware/mm_reflectometer/synth/mm_synth/active_bias.kicad_sch (KiCad schematic)
At the start: 23 parts

Commit message: added dac to mm_synth for vtune/adjstable bias, added ADC for telemetry
Connections:
- net +5V is gone; now on net +5VA: R?.1
Changed lines of the file:
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@@
     (pin "1")
   )
-  (symbol (lib_id "power:+5V") (at 177.8 46.99 0) (unit 1)
+  (symbol (lib_id "power:+5VA") (at 177.8 46.99 0) (unit 1)
     (in_bom yes) (on_board yes)
     (property "Reference" "#PWR?" (id 0) (at 177.8 50.8 0)
       (effects (font (size 1.27 1.27)) hide)
     )
-    (property "Value" "+5V" (id 1) (at 179.07 41.91 0))
+    (property "Value" "+5VA" (id 1) (at 179.07 41.91 0))
     (property "Footprint" "" (id 2) (at 177.8 46.99 0)
       (effects (font (size 1.27 1.27)) hide)

Commit message: work on mm synth schematic - control signals and footprint assignments
Parts:
- gave numbers to parts that had none: 23

Commit message: added usb PD sink to synth
Parts:
- added D1204: BAS516, Diode_SMD:D_SOD-523, symbol Diode:BAS516
Changed lines of the file:
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@@
+    (pin "2")
+  )
+  (symbol (lib_id "Diode:BAS516") (at 161.4396 134.1338 270) (unit 1)
+    (in_bom yes) (on_board yes)
+    (property "Reference" "D1204" (id 0) (at 163.9796 132.8638 90)
+      (effects (font (size 1.27 1.27)) (justify left))
+    )
+    (property "Value" "BAS516" (id 1) (at 163.9796 135.4038 90)
+      (effects (font (size 1.27 1.27)) (justify left))
+    )
+    (property "Footprint" "Diode_SMD:D_SOD-523" (id 2) (at 156.9946 134.1338 0)
+      (effects (font (size 1.27 1.27)) hide)
+    )
+    (property "Datasheet" "https://assets.nexperia.com/documents/data-sheet/BAS16_SER.pdf" (id 3) (at 161.4396 134.1338 0)
+      (effects (font (size 1.27 1.27)) hide)
+    )
+    (pin "1")
     (pin "2")
   )

Commit message: created HUSB238 eval board, added clock splitter to mm synth
Parts:
- removed D1204: BAS516, Diode_SMD:D_SOD-523, symbol Diode:BAS516
Changed lines of the file:
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@@
   (symbol (lib_id "Device:R_Small") (at 121.92 125.73 90) (unit 1)
     (in_bom yes) (on_board yes)
-    (property "Reference" "R1201" (id 0) (at 121.92 119.38 90))
-    (property "Value" "15k" (id 1) (at 121.92 121.92 90))
+    (property "Reference" "R1201" (id 0) (at 121.92 123.19 90))
+    (property "Value" "15k" (id 1) (at 121.92 128.27 90))
     (property "Footprint" "Resistor_SMD:R_0402_1005Metric" (id 2) (at 121.92 125.73 0)
       (effects (font (size 1.27 1.27)) hide)
@@
   (symbol (lib_id "Device:R_Small") (at 125.73 110.49 180) (unit 1)
     (in_bom yes) (on_board yes)
-    (property "Reference" "R1202" (id 0) (at 123.19 109.22 0))
-    (property "Value" "DNI" (id 1) (at 123.19 111.76 0))
+    (property "Reference" "R1202" (id 0) (at 130.81 110.49 0))
+    (property "Value" "DNI" (id 1) (at 129.54 113.03 0))
     (property "Footprint" "Resistor_SMD:R_0402_1005Metric" (id 2) (at 125.73 110.49 0)
       (effects (font (size 1.27 1.27)) hide)
@@
   (symbol (lib_id "Device:R_Small") (at 130.81 105.41 270) (unit 1)
     (in_bom yes) (on_board yes)
-    (property "Reference" "R1204" (id 0) (at 129.54 107.95 0))
-    (property "Value" "0" (id 1) (at 132.08 107.95 0))
+    (property "Reference" "R1204" (id 0) (at 132.08 102.87 90))
+    (property "Value" "0" (id 1) (at 129.54 107.95 90))
     (property "Footprint" "Resistor_SMD:R_0402_1005Metric" (id 2) (at 130.81 105.41 0)
       (effects (font (size 1.27 1.27)) hide)
@@
   (symbol (lib_id "Device:R_Small") (at 149.86 125.73 90) (unit 1)
     (in_bom yes) (on_board yes)
-    (property "Reference" "R1205" (id 0) (at 149.86 119.38 90))
-    (property "Value" "1k" (id 1) (at 149.86 121.92 90))
+    (property "Reference" "R1205" (id 0) (at 149.86 123.19 90))
+    (property "Value" "1k" (id 1) (at 149.86 128.27 90))
     (property "Footprint" "Resistor_SMD:R_0402_1005Metric" (id 2) (at 149.86 125.73 0)
       (effects (font (size 1.27 1.27)) hide)
@@
   (symbol (lib_id "Device:R_Small") (at 152.4 76.2 0) (unit 1)
     (in_bom yes) (on_board yes)
-    (property "Reference" "R1206" (id 0) (at 154.94 74.93 0)
-      (effects (font (size 1.27 1.27)) (justify left))
-    )
-    (property "Value" "1k" (id 1) (at 154.94 77.47 0)
+    (property "Reference" "R1206" (id 0) (at 144.78 74.93 0)
+      (effects (font (size 1.27 1.27)) (justify left))
+    )
+    (property "Value" "1k" (id 1) (at 148.59 77.47 0)
       (effects (font (size 1.27 1.27)) (justify left))
     )
@@
   (symbol (lib_id "Device:C_Small") (at 93.98 76.2 0) (unit 1)
     (in_bom yes) (on_board yes)
-    (property "Reference" "C1201" (id 0) (at 96.52 74.93 0)
-      (effects (font (size 1.27 1.27)) (justify left))
-    )
-    (property "Value" "100 pF" (id 1) (at 96.52 77.47 0)
+    (property "Reference" "C1201" (id 0) (at 95.25 74.93 0)
+      (effects (font (size 1.27 1.27)) (justify left))
+    )
+    (property "Value" "100 pF" (id 1) (at 95.25 78.74 0)
       (effects (font (size 1.27 1.27)) (justify left))
     )
@@
   (symbol (lib_id "Device:C_Small") (at 105.41 76.2 0) (unit 1)
     (in_bom yes) (on_board yes)
-    (property "Reference" "C1203" (id 0) (at 107.95 74.93 0)
-      (effects (font (size 1.27 1.27)) (justify left))
-    )
-    (property "Value" "100 nF" (id 1) (at 107.95 77.47 0)
+    (property "Reference" "C1203" (id 0) (at 106.68 74.93 0)
+      (effects (font (size 1.27 1.27)) (justify left))
+    )
+    (property "Value" "100 nF" (id 1) (at 106.68 78.74 0)
       (effects (font (size 1.27 1.27)) (justify left))
     )
@@
   (symbol (lib_id "Device:C_Small") (at 115.57 76.2 0) (unit 1)
     (in_bom yes) (on_board yes)
-    (property "Reference" "C1205" (id 0) (at 118.11 74.93 0)
-      (effects (font (size 1.27 1.27)) (justify left))
-    )
-    (property "Value" "4.7 uF" (id 1) (at 118.11 77.47 0)
+    (property "Reference" "C1205" (id 0) (at 116.84 74.93 0)
+      (effects (font (size 1.27 1.27)) (justify left))
+    )
+    (property "Value" "4.7 uF" (id 1) (at 116.84 78.74 0)
       (effects (font (size 1.27 1.27)) (justify left))
     )
@@
     (pin "2")
   )
-  (symbol (lib_id "Diode:BAS516") (at 161.4396 134.1338 270) (unit 1)
-    (in_bom yes) (on_board yes)
-    (property "Reference" "D1204" (id 0) (at 163.9796 132.8638 90)
-      (effects (font (size 1.27 1.27)) (justify left))
-    )
-    (property "Value" "BAS516" (id 1) (at 163.9796 135.4038 90)
-      (effects (font (size 1.27 1.27)) (justify left))
-    )
-    (property "Footprint" "Diode_SMD:D_SOD-523" (id 2) (at 156.9946 134.1338 0)
-      (effects (font (size 1.27 1.27)) hide)
-    )
-    (property "Datasheet" "https://assets.nexperia.com/documents/data-sheet/BAS16_SER.pdf" (id 3) (at 161.4396 134.1338 0)
-      (effects (font (size 1.27 1.27)) hide)
-    )
-    (pin "1")
-    (pin "2")
-  )
   (symbol (lib_id "Amplifier_Operational:TLV9001IDCK") (at 154.94 86.36 90) (mirror x) (unit 1)
     (in_bom yes) (on_board yes)
-    (property "Reference" "U1201" (id 0) (at 139.7 80.01 90)
-      (effects (font (size 1.27 1.27)) (justify left))
-    )
-    (property "Value" "TLV9151IDCKR" (id 1) (at 149.86 77.47 90)
-      (effects (font (size 1.27 1.27)) (justify left))
-    )
+    (property "Reference" "U1201" (id 0) (at 148.59 83.82 90)
+      (effects (font (size 1.27 1.27)) (justify left))
+    )
+    (property "Value" "TLV9151IDCKR" (id 1) (at 148.59 81.28 90)
+      (effects (font (size 1.27 1.27)) (justify left))
+    )
