File: hardware/mm_reflectometer/synth/mm_synth/synth.kicad_sch (KiCad schematic)
At the start: 46 parts, among them U201 VEMI65AB-HCI, U202 LMX2820

Commit message: created HUSB238 eval board, added clock splitter to mm synth
Parts:
- added R209: 100, Resistor_SMD:R_0402_1005Metric, symbol Device:R_Small
- R201, R202: value 50 -> DNI
Connections:
- net OSCIN_N: now also R209.2
- net OSCIN_P: now also R209.1
Changed lines of the file:
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@@
   (paper "A4")
   (junction (at 64.77 102.87) (diameter 0.9144) (color 0 0 0 0))
+  (junction (at 73.66 102.87) (diameter 0.9144) (color 0 0 0 0))
   (junction (at 73.66 110.49) (diameter 0.9144) (color 0 0 0 0))
   (junction (at 86.36 31.75) (diameter 0.9144) (color 0 0 0 0))
@@
     (stroke (width 0) (type solid) (color 0 0 0 0))
   )
+  (wire (pts (xy 73.66 102.87) (xy 64.77 102.87))
+    (stroke (width 0) (type solid) (color 0 0 0 0))
+  )
+  (wire (pts (xy 73.66 102.87) (xy 73.66 104.14))
+    (stroke (width 0) (type solid) (color 0 0 0 0))
+  )
+  (wire (pts (xy 73.66 109.22) (xy 73.66 110.49))
+    (stroke (width 0) (type solid) (color 0 0 0 0))
+  )
   (wire (pts (xy 73.66 110.49) (xy 73.66 111.76))
     (stroke (width 0) (type solid) (color 0 0 0 0))
@@
     (stroke (width 0) (type solid) (color 0 0 0 0))
   )
-  (wire (pts (xy 87.63 102.87) (xy 64.77 102.87))
+  (wire (pts (xy 87.63 102.87) (xy 73.66 102.87))
     (stroke (width 0) (type solid) (color 0 0 0 0))
   )
@@
     (in_bom yes) (on_board yes)
     (property "Reference" "R201" (id 0) (at 67.31 114.3 90))
-    (property "Value" "50" (id 1) (at 62.23 114.3 90))
+    (property "Value" "DNI" (id 1) (at 62.23 114.3 90))
     (property "Footprint" "Resistor_SMD:R_0402_1005Metric" (id 2) (at 64.77 114.3 0)
       (effects (font (size 1.27 1.27)) hide)
@@
     (pin "2")
   )
+  (symbol (lib_id "Device:R_Small") (at 73.66 106.68 0) (unit 1)
+    (in_bom yes) (on_board yes)
+    (property "Reference" "R209" (id 0) (at 76.2 106.68 90))
+    (property "Value" "100" (id 1) (at 71.12 106.68 90))
+    (property "Footprint" "Resistor_SMD:R_0402_1005Metric" (id 2) (at 73.66 106.68 0)
+      (effects (font (size 1.27 1.27)) hide)
+    )
+    (property "Datasheet" "~" (id 3) (at 73.66 106.68 0)
+      (effects (font (size 1.27 1.27)) hide)
+    )
+    (pin "1")
+    (pin "2")
+  )
   (symbol (lib_id "Device:R_Small") (at 73.66 114.3 0) (unit 1)
     (in_bom yes) (on_board yes)
     (property "Reference" "R202" (id 0) (at 76.2 114.3 90))
-    (property "Value" "50" (id 1) (at 71.12 114.3 90))
+    (property "Value" "DNI" (id 1) (at 71.12 114.3 90))
     (property "Footprint" "Resistor_SMD:R_0402_1005Metric" (id 2) (at 73.66 114.3 0)
       (effects (font (size 1.27 1.27)) hide)

Commit message: commit mm_synth prior to updating from june to september kicad-nightly build
Parts:
- C227: footprint Capacitor_SMD:C_0603_1608Metric -> Capacitor_SMD:C_1206_3216Metric
Changed lines of the file:
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@@
   (symbol (lib_id "Device:C_Small") (at 210.82 142.24 0) (unit 1)
     (in_bom yes) (on_board yes)
-    (property "Reference" "C225" (id 0) (at 214.63 142.24 0))
+    (property "Reference" "C225" (id 0) (at 215.9 142.24 0))
     (property "Value" "470 pF" (id 1) (at 215.9 144.78 0))
     (property "Footprint" "Capacitor_SMD:C_0603_1608Metric" (id 2) (at 210.82 142.24 0)
@@
   (symbol (lib_id "Device:C_Small") (at 222.25 142.24 0) (unit 1)
     (in_bom yes) (on_board yes)
-    (property "Reference" "C227" (id 0) (at 226.06 142.24 0))
+    (property "Reference" "C227" (id 0) (at 227.33 142.24 0))
     (property "Value" "68 nF" (id 1) (at 227.33 144.78 0))
-    (property "Footprint" "Capacitor_SMD:C_0603_1608Metric" (id 2) (at 222.25 142.24 0)
+    (property "Footprint" "Capacitor_SMD:C_1206_3216Metric" (id 2) (at 222.25 142.24 0)
       (effects (font (size 1.27 1.27)) hide)
     )
@@
   (symbol (lib_id "Device:C_Small") (at 236.22 142.24 0) (unit 1)
     (in_bom yes) (on_board yes)
-    (property "Reference" "C229" (id 0) (at 240.03 142.24 0))
+    (property "Reference" "C229" (id 0) (at 241.3 142.24 0))
     (property "Value" "2.2 nF" (id 1) (at 241.3 144.78 0))
     (property "Footprint" "Capacitor_SMD:C_0603_1608Metric" (id 2) (at 236.22 142.24 0)
