File: breakouts/bias_controller/bias_controller/load_switch.kicad_sch (KiCad schematic)
At the start: 7 parts, among them U11 INA199B1DCKR, U12 TPS22917DBV, U13 TPS22917DBV

Commit message: bias controller schematic work
Parts:
- added C29, C30: 100 pF, symbol Device:C_Small
- added R49, R50: 0, symbol Device:R_Small
Connections:
- net +3.3VP: now also U13.1 (VIN), C30.1
- net 3V3_SWITCHED: now also U13.6 (VOUT), R50.1
- net GND: now also U12.2 (GND), U13.2 (GND)
- net at R47.1, U11.4 (+): now also U12.6 (VOUT), R49.1
- net 3V3_SW_EN: now reaches U13.3 (ON)
- net at U13.4 (CT): now also C30.2
- net at U13.5 (QOD): now also R50.2
- net VDD: now reaches U12.1 (VIN)
- net VDD: now also C29.1
- net VDD_SW_EN: now reaches U12.3 (ON)
- net at U12.4 (CT): now also C29.2
- net at U12.5 (QOD): now also R49.2
Other:
- moved on the sheet: U12

Commit message: top level schematic work
Parts:
- renumbered C29 to C27, C30 to C28, C28 to C29, C27 to C30, R49 to R47, R50 to R48, R47 to R49, R48 to R50, U12 to U11, U13 to U12, U11 to U13
Changed lines of the file:
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@@
   (symbol (lib_id "Device:R_Small") (at 149.86 116.84 0) (unit 1)
     (exclude_from_sim no) (in_bom yes) (on_board yes) (dnp no) (fields_autoplaced)
-    (property "Reference" "R50" (at 152.4 115.5699 0)
+    (property "Reference" "R48" (at 152.4 115.5699 0)
       (effects (font (size 1.27 1.27)) (justify left))
     )
@@
   (symbol (lib_id "power:GND") (at 130.81 124.46 0) (unit 1)
     (exclude_from_sim no) (in_bom yes) (on_board yes) (dnp no) (fields_autoplaced)
-    (property "Reference" "#PWR072" (at 130.81 130.81 0)
+    (property "Reference" "#PWR067" (at 130.81 130.81 0)
       (effects (font (size 1.27 1.27)) hide)
     )
@@
   (symbol (lib_id "Device:C_Small") (at 198.12 43.18 0) (unit 1)
     (exclude_from_sim no) (in_bom yes) (on_board yes) (dnp no) (fields_autoplaced)
-    (property "Reference" "C28" (at 200.66 41.9163 0)
+    (property "Reference" "C29" (at 200.66 41.9163 0)
       (effects (font (size 1.27 1.27)) (justify left))
     )
@@
   (symbol (lib_id "power:GND") (at 209.55 66.04 0) (unit 1)
     (exclude_from_sim no) (in_bom yes) (on_board yes) (dnp no) (fields_autoplaced)
-    (property "Reference" "#PWR066" (at 209.55 72.39 0)
+    (property "Reference" "#PWR070" (at 209.55 72.39 0)
       (effects (font (size 1.27 1.27)) hide)
     )
@@
   (symbol (lib_id "Device:R_Small") (at 193.04 57.15 0) (unit 1)
     (exclude_from_sim no) (in_bom yes) (on_board yes) (dnp no) (fields_autoplaced)
-    (property "Reference" "R47" (at 195.58 55.88 0)
+    (property "Reference" "R49" (at 195.58 55.88 0)
       (effects (font (size 1.27 1.27)) (justify left))
     )
@@
   (symbol (lib_id "Power_Management:TPS22917DBV") (at 130.81 114.3 0) (unit 1)
     (exclude_from_sim no) (in_bom yes) (on_board yes) (dnp no) (fields_autoplaced)
-    (property "Reference" "U13" (at 130.81 104.14 0)
+    (property "Reference" "U12" (at 130.81 104.14 0)
       (effects (font (size 1.27 1.27)))
     )
@@
   (symbol (lib_id "Device:R_Small") (at 149.86 41.91 0) (unit 1)
     (exclude_from_sim no) (in_bom yes) (on_board yes) (dnp no) (fields_autoplaced)
-    (property "Reference" "R49" (at 152.4 40.6399 0)
+    (property "Reference" "R47" (at 152.4 40.6399 0)
       (effects (font (size 1.27 1.27)) (justify left))
     )
@@
   (symbol (lib_id "power:GND") (at 228.6 73.66 0) (unit 1)
     (exclude_from_sim no) (in_bom yes) (on_board yes) (dnp no) (fields_autoplaced)
-    (property "Reference" "#PWR067" (at 228.6 80.01 0)
+    (property "Reference" "#PWR072" (at 228.6 80.01 0)
       (effects (font (size 1.27 1.27)) hide)
     )
@@
   (symbol (lib_id "Amplifier_Current:INA199xxDCK") (at 212.09 57.15 0) (unit 1)
     (exclude_from_sim no) (in_bom yes) (on_board yes) (dnp no)
-    (property "Reference" "U11" (at 215.9 49.53 0)
+    (property "Reference" "U13" (at 215.9 49.53 0)
       (effects (font (size 1.27 1.27)))
     )
@@
   (symbol (lib_id "power:GND") (at 130.81 49.53 0) (unit 1)
     (exclude_from_sim no) (in_bom yes) (on_board yes) (dnp no) (fields_autoplaced)
-    (property "Reference" "#PWR070" (at 130.81 55.88 0)
+    (property "Reference" "#PWR066" (at 130.81 55.88 0)
       (effects (font (size 1.27 1.27)) hide)
     )
@@
   (symbol (lib_id "Device:C_Small") (at 110.49 119.38 90) (unit 1)
     (exclude_from_sim no) (in_bom yes) (on_board yes) (dnp no) (fields_autoplaced)
-    (property "Reference" "C30" (at 110.4963 113.03 90)
+    (property "Reference" "C28" (at 110.4963 113.03 90)
       (effects (font (size 1.27 1.27)))
     )
@@
   (symbol (lib_id "Power_Management:TPS22917DBV") (at 130.81 39.37 0) (unit 1)
     (exclude_from_sim no) (in_bom yes) (on_board yes) (dnp no) (fields_autoplaced)
-    (property "Reference" "U12" (at 130.81 29.21 0)
+    (property "Reference" "U11" (at 130.81 29.21 0)
       (effects (font (size 1.27 1.27)))
     )
@@
   (symbol (lib_id "Device:R_Small") (at 214.63 69.85 0) (unit 1)
     (exclude_from_sim no) (in_bom yes) (on_board yes) (dnp no) (fields_autoplaced)
-    (property "Reference" "R48" (at 217.17 68.58 0)
+    (property "Reference" "R50" (at 217.17 68.58 0)
       (effects (font (size 1.27 1.27)) (justify left))
     )
@@
   (symbol (lib_id "Device:C_Small") (at 228.6 69.85 0) (unit 1)
     (exclude_from_sim no) (in_bom yes) (on_board yes) (dnp no) (fields_autoplaced)
-    (property "Reference" "C27" (at 231.14 68.5863 0)
+    (property "Reference" "C30" (at 231.14 68.5863 0)
       (effects (font (size 1.27 1.27)) (justify left))
     )
@@
   (symbol (lib_id "Device:C_Small") (at 110.49 44.45 90) (unit 1)
     (exclude_from_sim no) (in_bom yes) (on_board yes) (dnp no) (fields_autoplaced)
-    (property "Reference" "C29" (at 110.4963 38.1 90)
-      (effects (font (size 1.27 1.27)))
-    )
+    (property "Reference" "C27" (at 110.4963 38.1 90)
+      (effects (font (size 1.27 1.27)))
+    )

Commit message: most footprint assignments on bias controller board, schematic cleanup
Parts:
- removed C30: 100 nF, symbol Device:C_Small
- C701: renamed from C27; footprint (none) -> Capacitor_SMD:C_0402_1005Metric
- C702: renamed from C28; footprint (none) -> Capacitor_SMD:C_0402_1005Metric
- C703: renamed from C29; footprint (none) -> Capacitor_SMD:C_0402_1005Metric
- R701: renamed from R47; footprint (none) -> Resistor_SMD:R_0402_1005Metric
- R702: renamed from R48; footprint (none) -> Resistor_SMD:R_0402_1005Metric
- R703: renamed from R49; value R_Small -> 0.05; footprint (none) -> Resistor_SMD:R_1206_3216Metric
- R704: renamed from R50; value R_Small -> 0; footprint (none) -> Resistor_SMD:R_1206_3216Metric
- renumbered U11 to U701, U12 to U702, U13 to U703
Connections:
- net +3.3VP: no longer R704.2
- net GND: now also R704.2

Commit message: added LCSC part numbers to all components on bias board
Parts:
- C701, C702: LCSC Part # (none) -> C1546
- C703: LCSC Part # (none) -> C307331
- R701, R702: LCSC Part # (none) -> C17168
- R703: LCSC Part # (none) -> C601088
- R704: footprint Resistor_SMD:R_1206_3216Metric -> Resistor_SMD:R_0402_1005Metric; LCSC Part # (none) -> C17168
- U701, U702: LCSC Part # (none) -> C2681320
- U703: LCSC Part # (none) -> C398920
Changed lines of the file:
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@@
 			)
 		)
-		(property "LCSC Part #" ""
+		(property "LCSC Part #" "C17168"
 			(at 149.86 116.84 0)
 			(effects
@@
 			)
 		)
-		(property "LCSC Part #" ""
+		(property "LCSC Part #" "C307331"
 			(at 198.12 43.18 0)
 			(effects
@@
 			)
 		)
-		(property "LCSC Part #" ""
+		(property "LCSC Part #" "C601088"
 			(at 193.04 57.15 0)
 			(effects
@@
 			)
 		)
-		(property "LCSC Part #" ""
+		(property "LCSC Part #" "C2681320"
 			(at 130.81 114.3 0)
 			(effects
@@
 			)
 		)
-		(property "LCSC Part #" ""
+		(property "LCSC Part #" "C17168"
 			(at 149.86 41.91 0)
 			(effects
@@
 			)
 		)
-		(property "LCSC Part #" ""
+		(property "LCSC Part #" "C398920"
 			(at 212.09 57.15 0)
 			(effects
@@
 			)
 		)
-		(property "LCSC Part #" ""
+		(property "LCSC Part #" "C1546"
 			(at 110.49 119.38 0)
 			(effects
@@
 			)
 		)
-		(property "LCSC Part #" ""
+		(property "LCSC Part #" "C2681320"
 			(at 130.81 39.37 0)
 			(effects
@@
 			)
 		)
-		(property "Footprint" "Resistor_SMD:R_1206_3216Metric"
+		(property "Footprint" "Resistor_SMD:R_0402_1005Metric"
 			(at 214.63 69.85 0)
 			(effects
@@
 			)
 		)
-		(property "LCSC Part #" ""
+		(property "LCSC Part #" "C17168"
 			(at 214.63 69.85 0)
 			(effects
@@
 			)
 		)
-		(property "LCSC Part #" ""
+		(property "LCSC Part #" "C1546"
 			(at 110.49 44.45 0)
 			(effects
